Commit message: Compute stereo point clouds from lander's camera. Adjusted optical frames so point clouds can be displayed in rviz in the proper locations.

File: ow_lander/urdf/stereo_camera_triggered.xacro (robot description, xacro)
@@ -62,5 +62,5 @@
   </joint>
   <joint name="leftCamera_optical_joint" type="fixed">
-    <origin xyz="0.0 0.0 0.0" rpy="0 0 0"/>
+    <origin xyz="0.0 0.0 0.0" rpy="-${pi/2} 0 -${pi/2}"/>
     <parent link="${Camera01Name}Left_link"/>
     <child link="${Camera01Name}Left_optical_frame"/>
@@ -75,5 +75,5 @@
   </joint>
   <joint name="rightCamera_optical_joint" type="fixed">
-    <origin xyz="0.0 0.0 0.0" rpy="0 0 0"/>
+    <origin xyz="0.0 0.0 0.0" rpy="-${pi/2} 0 -${pi/2}"/>
     <parent link="${Camera01Name}Right_link"/>
     <child link="${Camera01Name}Right_optical_frame"/>
@@ -138,5 +138,5 @@
   </joint>
   <joint name="CenterCamera_optical_joint" type="fixed">
-    <origin xyz="0.0 0.0 0.0" rpy="0 0 0"/>
+    <origin xyz="0.0 0.0 0.0" rpy="-${pi/2} 0 -${pi/2}"/>
     <parent link="${Camera01Name}Center_link"/>
     <child link="${Camera01Name}Center_optical_frame"/>

Commit message: Renamed NavCamStereo to StereoCamera.

File: ow_lander/urdf/stereo_camera_triggered.xacro (robot description, xacro)
@@ -1,5 +1,5 @@
 <?xml version="1.0"?>
 <robot xmlns:xacro="http://ros.org/wiki/xacro" name="stereo_camera">
-  <xacro:property name="Camera01Name"       value="NavCamStereo" />
+  <xacro:property name="Camera01Name"       value="StereoCamera" />
   <xacro:property name="Camera01UpdateRate" value="5" />
   <xacro:property name="camera_baseline"    value="0.2" />
