Commit message: Fixed sample dock collision box position.

File: ow_lander/urdf/lander_sample_dock.xacro (robot description, xacro)
@@ -21,5 +21,5 @@
     <link name="lander_sample_dock${suffix}">
       <collision>
-        <origin rpy="0 0 0" xyz="0 0 0.25"/>
+        <origin rpy="0 0 0" xyz="0 0 0.025"/>
         <geometry>
           <box size="0.3 0.05 0.095"/>

Commit message: A sample dock that can hold collected samples

File: ow_lander/urdf/lander_sample_dock.xacro (robot description, xacro)
@@ -26,5 +26,5 @@
         <origin rpy="0 0 0" xyz="0 0 0.025"/>
         <geometry>
-          <box size="0.3 0.05 0.095"/>
+          <mesh filename="package://ow_lander/meshes/sample_dock.stl" />
         </geometry>
       </collision>
@@ -32,5 +32,5 @@
         <origin rpy="0 0 0" xyz="0 0 0.025"/>
         <geometry>
-          <box size="0.3 0.05 0.095"/>
+          <mesh filename="package://ow_lander/meshes/sample_dock.stl" />
         </geometry>
         <material name="">
@@ -42,7 +42,7 @@
         <mass value="0.01"/>
         <inertia
-            ixx="${sample_dock_mass / 12.0 * (0.1*0.1 + 0.06*0.06)}" ixy="0.0" ixz="0.0"
-            iyy="${sample_dock_mass / 12.0 * (0.06*0.06 + 0.1*0.1)}" iyz="0.0"
-            izz="${sample_dock_mass / 12.0 * (0.06*0.06 + 0.06*0.06)}"/>
+            ixx="${sample_dock_mass * 0.000001}" ixy="0.0" ixz="0.0"
+            iyy="${sample_dock_mass * 0.000006}" iyz="0.0"
+            izz="${sample_dock_mass * 0.000006}"/>
       </inertial>
     </link>

Commit message: Sample dock blocked-out as box colliders instead of using STL mesh

File: ow_lander/urdf/lander_sample_dock.xacro (robot description, xacro)
@@ -23,8 +23,53 @@
   <xacro:macro name="lander_sample_dock_link" params="suffix roll pitch y">
     <link name="lander_sample_dock${suffix}">
-      <collision>
+      <!-- <collision>
         <origin rpy="0 0 0" xyz="0 0 0"/>
         <geometry>
           <mesh filename="package://ow_lander/meshes/sample_dock.stl" />
+        </geometry>
+      </collision> -->
+      <!-- dock bottom -->
+      <collision>
+        <origin
+          xyz="0 0.0197015 0"
+          rpy="0 0 0" />
+        <geometry>
+          <box size="0.3 0.010597 0.095"/>
+        </geometry>
+      </collision>
+      <!-- dock +z wall -->
+      <collision>
+        <origin
+          xyz="0 0 0.04275"
+          rpy="0 0 0" />
+        <geometry>
+          <box size="0.3 0.05 0.0095"/>
+        </geometry>
+      </collision>
+      <!-- dock -z wall -->
+      <collision>
+        <origin
+          xyz="0 0 -0.04275"
+          rpy="0 0 0" />
+        <geometry>
+          <box size="0.3 0.05 0.0095"/>
+        </geometry>
+      </collision>
+      <!-- dock +x wall -->
+      <collision>
+        <origin
+          xyz="0.1425 0 0"
+          rpy="0 0 0" />
+        <geometry>
+          <box size="0.015 0.05 0.095"/>
+        </geometry>
+      </collision>
+      <!-- dock -x wall -->
+      <collision>
+        <origin
+          xyz="-0.1425 0 0"
+          rpy="0 0 0" />
+        <geometry>
+          <box size="0.015 0.05 0.095"/>
         </geometry>
       </collision>

Commit message: Removed commented-out lines

File: ow_lander/urdf/lander_sample_dock.xacro (robot description, xacro)
@@ -23,10 +23,4 @@
   <xacro:macro name="lander_sample_dock_link" params="suffix roll pitch y">
     <link name="lander_sample_dock${suffix}">
-      <!-- <collision>
-        <origin rpy="0 0 0" xyz="0 0 0"/>
-        <geometry>
-          <mesh filename="package://ow_lander/meshes/sample_dock.stl" />
-        </geometry>
-      </collision> -->
       <!-- dock bottom -->
       <collision>

Commit message: rebuilt DockIngestSample to now look at positions itself

File: ow_lander/urdf/lander_sample_dock.xacro (robot description, xacro)
@@ -63,17 +63,4 @@
         </plugin>
       </visual>
-      <sensor name="contact_sensor_sample_dock" type="contact">
-        <parent link="lander_sample_dock${suffix}"/>
-        <contact>
-          <collision>
-            lander_sample_dock_link_fixed_joint_lump__lander_sample_dock${suffix}_collision
-          </collision>
-        </contact>
-        <plugin name="contact_sensor_sample_dock_plugin"
-                filename="libContactSensorPlugin.so">
-          <topic>/ow_regolith/contacts/sample_dock</topic>
-          <report_only>regolith_\d*.*</report_only>
-        </plugin>
-      </sensor>
     </gazebo>
   </xacro:macro>
