Commit message: Updated lander model.

File: ow_lander/urdf/lander.xacro (robot description, xacro)
@@ -11,497 +11,381 @@
     <inertial>
       <origin
-        xyz="-0.174891183141199 0.105186140838806 0.499102801889294"
-        rpy="0 0 0" />
-      <mass
-        value="921.409320871089" />
-      <inertia
-        ixx="33.2402321826437"
-        ixy="0.60557675951993"
-        ixz="-0.0951190939564292"
-        iyy="33.9643287034463"
-        iyz="0.0499080883396483"
-        izz="63.3487609623066" />
-    </inertial>
-    <visual>
-      <origin
-        xyz="0 0 0"
-        rpy="0 0 0" />
-      <geometry>
-        <mesh
-          filename="package://ow_lander/meshes/lander_body.STL" />
-      </geometry>
-      <material
-        name="">
-        <color
-          rgba="0.2 0.2 0.2 1" />
-      </material>
-    </visual>
-    <collision>
-      <origin
-        xyz="0 0 0"
-        rpy="0 0 0" />
-      <geometry>
-        <mesh
-          filename="package://ow_lander/meshes/lander_body.STL" />
-      </geometry>
-    </collision>
-  </link>
-  <link
-    name="link_shoulder">
-    <inertial>
-      <origin
-        xyz="0.0560579395709874 0.141768391065364 0.00404480198837498"
-        rpy="0 0 0" />
-      <mass
-        value="6.82139097144578" />
-      <inertia
-        ixx="0.00893744641566868"
-        ixy="0.00781896786597782"
-        ixz="-0.00236278992626154"
-        iyy="0.0275545990944527"
-        iyz="0.000600617787047249"
-        izz="0.0360781788843499" />
-    </inertial>
-    <visual>
-      <origin
-        xyz="0 0 0"
-        rpy="0 0 0" />
-      <geometry>
-        <mesh
-          filename="package://ow_lander/meshes/link_shoulder.STL" />
-      </geometry>
-      <material
-        name="">
-        <color
-          rgba="0.898039215686275 0.917647058823529 0.929411764705882 1" />
-      </material>
-    </visual>
-    <collision>
-      <origin
-        xyz="0 0 0"
-        rpy="0 0 0" />
-      <geometry>
-        <mesh
-          filename="package://ow_lander/meshes/link_shoulder.STL" />
-      </geometry>
-    </collision>
-  </link>
-  <joint
-    name="joint_shoulder_yaw"
-    type="continuous">
-    <origin
-      xyz="0.504875558700385 -0.329105217556347 0.325000000000001"
-      rpy="1.5707963267949 2.74973548348948E-17 0.46573620389147" />
+        xyz="0.002242 0.0014227 0.3241"
+        rpy="0 0 0" />
+      <mass
+        value="921.41" />
+      <inertia
+        ixx="32.997"
+        ixy="-0.36205"
+        ixz="-0.10255"
+        iyy="34.208"
+        iyz="-0.031969"
+        izz="63.349" />
+    </inertial>
+    <visual>
+      <origin
+        xyz="0 0 0"
+        rpy="0 0 0" />
+      <geometry>
+        <mesh
+          filename="package://ow_lander/meshes/base_link.STL" />
+      </geometry>
+      <material
+        name="">
+        <color
+          rgba="0.79216 0.81961 0.93333 1" />
+      </material>
+    </visual>
+    <collision>
+      <origin
+        xyz="0 0 0"
+        rpy="0 0 0" />
+      <geometry>
+        <mesh
+          filename="package://ow_lander/meshes/base_link.STL" />
+      </geometry>
+    </collision>
+  </link>
+  <link
+    name="l_shou">
+    <inertial>
+      <origin
+        xyz="0.0591309542444923 0.00156004002922039 -0.0211248119973624"
+        rpy="0 0 0" />
+      <mass
+        value="7.02920774782214" />
+      <inertia
+        ixx="0.0104575300282247"
+        ixy="-0.000601021251095754"
+        ixz="-0.00827528301657843"
+        iyy="0.0383526039269065"
+        iyz="-0.000231653878395009"
+        izz="0.0311579762615783" />
+    </inertial>
+    <visual>
+      <origin
+        xyz="0 0 0"
+        rpy="0 0 0" />
+      <geometry>
+        <mesh
+          filename="package://ow_lander/meshes/l_shou.STL" />
+      </geometry>
+      <material
+        name="">
+        <color
+          rgba="0.898039215686275 0.917647058823529 0.929411764705882 1" />
+      </material>
+    </visual>
+    <collision>
+      <origin
+        xyz="0 0 0"
+        rpy="0 0 0" />
+      <geometry>
+        <mesh
+          filename="package://ow_lander/meshes/l_shou.STL" />
+      </geometry>
+    </collision>
+  </link>
+  <joint
+    name="j_shou_yaw"
+    type="continuous">
+    <origin
+      xyz="0.79 0.175 0.27"
+      rpy="-3.1416 0 0" />
     <parent
       link="base_link" />
     <child
-      link="link_shoulder" />
-    <axis
-      xyz="0 1 0" />
-  </joint>
-  <transmission name="shoulder_yaw_transmission">
-    <type>transmission_interface/SimpleTransmission</type>
-    <joint name="joint_shoulder_yaw">
-      <hardwareInterface>hardware_interface/EffortJointInterface</hardwareInterface>
-    </joint>
-    <actuator name="shoulder_yaw_motor">
-      <mechanicalReduction>1</mechanicalReduction>
-    </actuator>
-  </transmission>
-  <link
-    name="link_proximal">
-    <inertial>
-      <origin
-        xyz="-0.0492100785879154 0.13596231010573 -0.00264198593257192"
-        rpy="0 0 0" />
-      <mass
-        value="4.19334465872563" />
-      <inertia
-        ixx="0.0984810896192592"
-        ixy="0.0219047703464202"
-        ixz="-0.000425647279922649"
-        iyy="0.0113852386512403"
-        iyz="0.00191279732232413"
-        izz="0.109791995726008" />
-    </inertial>
-    <visual>
-      <origin
-        xyz="0 0 0"
-        rpy="0 0 0" />
-      <geometry>
-        <mesh
-          filename="package://ow_lander/meshes/link_proximal.STL" />
-      </geometry>
-      <material
-        name="">
-        <color
-          rgba="0.898039215686275 0.917647058823529 0.929411764705882 1" />
-      </material>
-    </visual>
-    <collision>
-      <origin
-        xyz="0 0 0"
-        rpy="0 0 0" />
-      <geometry>
-        <mesh
-          filename="package://ow_lander/meshes/link_proximal.STL" />
-      </geometry>
-    </collision>
-  </link>
-  <joint
-    name="joint_shoulder_pitch"
-    type="continuous">
-    <origin
-      xyz="0.160000000000006 0.119999999999994 0.0549999999999998"
-      rpy="-3.07263964126294 1.57079630572147 -3.07263964126294" />
-    <parent
-      link="link_shoulder" />
-    <child
-      link="link_proximal" />
-    <axis
-      xyz="-1 0 0" />
-  </joint>
-  <transmission name="shoulder_pitch_transmission">
-    <type>transmission_interface/SimpleTransmission</type>
-    <joint name="joint_shoulder_pitch">
-      <hardwareInterface>hardware_interface/EffortJointInterface</hardwareInterface>
-    </joint>
-    <actuator name="shoulder_pitch_motor">
-      <mechanicalReduction>1</mechanicalReduction>
-    </actuator>
-  </transmission>
-  <link
-    name="link_distal">
-    <inertial>
-      <origin
-        xyz="-0.0270676297110266 1.19266541087626E-09 0.215098268051955"
-        rpy="0 0 0" />
-      <mass
-        value="7.67831405851241" />
-      <inertia
-        ixx="0.448007770505405"
-        ixy="3.27562144075699E-11"
-        ixz="0.0217064684901283"
-        iyy="0.456482852663482"
-        iyz="-7.1993979908723E-08"
-        izz="0.00847508215811156" />
-    </inertial>
-    <visual>
-      <origin
-        xyz="0 0 0"
-        rpy="0 0 0" />
-      <geometry>
-        <mesh
-          filename="package://ow_lander/meshes/link_distal.STL" />
-      </geometry>
-      <material
-        name="">
-        <color
-          rgba="0.898039215686275 0.917647058823529 0.929411764705882 1" />
-      </material>
-    </visual>
-    <collision>
-      <origin
-        xyz="0 0 0"
-        rpy="0 0 0" />
-      <geometry>
-        <mesh
-          filename="package://ow_lander/meshes/link_distal.STL" />
-      </geometry>
-    </collision>
-  </link>
-  <joint
-    name="joint_proximal_pitch"
-    type="continuous">
-    <origin
-      xyz="0 0.52989996780278 -0.0102968015714265"
-      rpy="-2.4583426132036 -5.55111512312578E-17 -3.14159265358979" />
-    <parent
-      link="link_proximal" />
-    <child
-      link="link_distal" />
-    <axis
-      xyz="1 0 0" />
-  </joint>
-  <transmission name="proximal_pitch_transmission">
-    <type>transmission_interface/SimpleTransmission</type>
-    <joint name="joint_proximal_pitch">
-      <hardwareInterface>hardware_interface/EffortJointInterface</hardwareInterface>
-    </joint>
-    <actuator name="proximal_pitch_motor">
-      <mechanicalReduction>1</mechanicalReduction>
-    </actuator>
-  </transmission>
-  <link
-    name="link_wrist">
-    <inertial>
-      <origin
-        xyz="0.0598274983548339 -0.00683833441329951 -0.0773548039852737"
-        rpy="0 0 0" />
-      <mass
-        value="4.03473451988803" />
-      <inertia
-        ixx="0.0233350554047849"
-        ixy="0.000832485639475045"
-        ixz="0.00924084473050794"
-        iyy="0.0271779846566029"
-        iyz="-0.00229121026195695"
-        izz="0.00433425186366915" />
-    </inertial>
-    <visual>
-      <origin
-        xyz="0 0 0"
-        rpy="0 0 0" />
-      <geometry>
-        <mesh
-          filename="package://ow_lander/meshes/link_wrist.STL" />
-      </geometry>
-      <material
-        name="">
-        <color
-          rgba="0.898039215686275 0.917647058823529 0.929411764705882 1" />
-      </material>
-    </visual>
-    <collision>
-      <origin
-        xyz="0 0 0"
-        rpy="0 0 0" />
-      <geometry>
-        <mesh
-          filename="package://ow_lander/meshes/link_wrist.STL" />
-      </geometry>
-    </collision>
-  </link>
-  <joint
-    name="joint_distal_pitch"
-    type="continuous">
-    <origin
-      xyz="0.00500000000000056 0 0.586000000000023"
-      rpy="2.56643026615587 3.77475828372553E-15 1.94289029309402E-15" />
-    <parent
-      link="link_distal" />
-    <child
-      link="link_wrist" />
-    <axis
-      xyz="1 0 0" />
-  </joint>
-  <transmission name="distal_pitch_transmission">
-    <type>transmission_interface/SimpleTransmission</type>
-    <joint name="joint_distal_pitch">
-      <hardwareInterface>hardware_interface/EffortJointInterface</hardwareInterface>
-    </joint>
-    <actuator name="distal_pitch_motor">
-      <mechanicalReduction>1</mechanicalReduction>
-    </actuator>
-  </transmission>
-  <link
-    name="link_hand">
-    <inertial>
-      <origin
-        xyz="0.0559835529936636 0.00390822003474067 0.00225571287946436"
-        rpy="0 0 0" />
-      <mass
-        value="3.29341647546119" />
-      <inertia
-        ixx="0.000109355149428239"
-        ixy="-0.000992165341035474"
-        ixz="-0.000572649471646507"
-        iyy="0.0168063828016295"
-        iyz="-4.73448318734377E-05"
-        izz="0.0168610857840526" />
-    </inertial>
-    <visual>
-      <origin
-        xyz="0 0 0"
-        rpy="0 0 0" />
-      <geometry>
-        <mesh
-          filename="package://ow_lander/meshes/link_hand.STL" />
-      </geometry>
-      <material
-        name="">
-        <color
-          rgba="0.898039215686275 0.917647058823529 0.929411764705882 1" />
-      </material>
-    </visual>
-    <collision>
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
Commit message: Added effort controllers that take position inputs to the arm and antenna. If we disable dynamics, we will want to change these to position or velocity controllers.

File: ow_lander/urdf/lander.xacro (robot description, xacro)
@@ -99,5 +99,15 @@
     <axis
       xyz="0 0 -1" />
-  </joint>
+    <dynamics damping="50" />
+  </joint>
+  <transmission name="shou_yaw_transmission">
+    <type>transmission_interface/SimpleTransmission</type>
+    <joint name="j_shou_yaw">
+      <hardwareInterface>hardware_interface/EffortJointInterface</hardwareInterface>
+    </joint>
+    <actuator name="shou_yaw_motor">
+      <mechanicalReduction>1</mechanicalReduction>
+    </actuator>
+  </transmission>
   <link
     name="l_prox">
@@ -152,5 +162,15 @@
     <axis
       xyz="0 0 -1" />
-  </joint>
+    <dynamics damping="50" />
+  </joint>
+  <transmission name="shou_pitch_transmission">
+    <type>transmission_interface/SimpleTransmission</type>
+    <joint name="j_shou_pitch">
+      <hardwareInterface>hardware_interface/EffortJointInterface</hardwareInterface>
+    </joint>
+    <actuator name="shou_pitch_motor">
+      <mechanicalReduction>1</mechanicalReduction>
+    </actuator>
+  </transmission>
   <link
     name="l_dist">
@@ -205,5 +225,15 @@
     <axis
       xyz="0 0 -1" />
-  </joint>
+    <dynamics damping="50" />
+  </joint>
+  <transmission name="prox_pitch_transmission">
+    <type>transmission_interface/SimpleTransmission</type>
+    <joint name="j_prox_pitch">
+      <hardwareInterface>hardware_interface/EffortJointInterface</hardwareInterface>
+    </joint>
+    <actuator name="prox_pitch_motor">
+      <mechanicalReduction>1</mechanicalReduction>
+    </actuator>
+  </transmission>
   <link
     name="l_wrist">
@@ -258,5 +288,15 @@
     <axis
       xyz="0 0 1" />
-  </joint>
+    <dynamics damping="50" />
+  </joint>
+  <transmission name="dist_pitch_transmission">
+    <type>transmission_interface/SimpleTransmission</type>
+    <joint name="j_dist_pitch">
+      <hardwareInterface>hardware_interface/EffortJointInterface</hardwareInterface>
+    </joint>
+    <actuator name="dist_pitch_motor">
+      <mechanicalReduction>1</mechanicalReduction>
+    </actuator>
+  </transmission>
   <link
     name="l_hand">
@@ -311,5 +351,15 @@
     <axis
       xyz="0 0 -1" />
-  </joint>
+    <dynamics damping="50" />
+  </joint>
+  <transmission name="hand_yaw_transmission">
+    <type>transmission_interface/SimpleTransmission</type>
+    <joint name="j_hand_yaw">
+      <hardwareInterface>hardware_interface/EffortJointInterface</hardwareInterface>
+    </joint>
+    <actuator name="hand_yaw_motor">
+      <mechanicalReduction>1</mechanicalReduction>
+    </actuator>
+  </transmission>
   <link
     name="l_scoop">
@@ -364,5 +414,15 @@
     <axis
       xyz="0 0 -1" />
-  </joint>
+    <dynamics damping="50" />
+  </joint>
+  <transmission name="scoop_yaw_transmission">
+    <type>transmission_interface/SimpleTransmission</type>
+    <joint name="j_scoop_yaw">
+      <hardwareInterface>hardware_interface/EffortJointInterface</hardwareInterface>
+    </joint>
+    <actuator name="scoop_yaw_motor">
+      <mechanicalReduction>1</mechanicalReduction>
+    </actuator>
+  </transmission>
   <link
     name="l_ant_foot">
@@ -417,5 +477,15 @@
     <axis
       xyz="0 0 -1" />
-  </joint>
+    <dynamics damping="50" />
+  </joint>
+  <transmission name="ant_pan_transmission">
+    <type>transmission_interface/SimpleTransmission</type>
+    <joint name="j_ant_pan">
+      <hardwareInterface>hardware_interface/EffortJointInterface</hardwareInterface>
+    </joint>
+    <actuator name="ant_pan_motor">
+      <mechanicalReduction>1</mechanicalReduction>
+    </actuator>
+  </transmission>
   <link
     name="l_ant_panel">
@@ -470,15 +540,25 @@
     <axis
       xyz="0 0 -1" />
-  </joint>
+    <dynamics damping="50" />
+  </joint>
+  <transmission name="ant_tilt_transmission">
+    <type>transmission_interface/SimpleTransmission</type>
+    <joint name="j_ant_tilt">
+      <hardwareInterface>hardware_interface/EffortJointInterface</hardwareInterface>
+    </joint>
+    <actuator name="ant_tilt_motor">
+      <mechanicalReduction>1</mechanicalReduction>
+    </actuator>
+  </transmission>
   <gazebo>
-    <!--plugin name="gazebo_ros_control" filename="libgazebo_ros_control.so">
+    <plugin name="gazebo_ros_control" filename="libgazebo_ros_control.so">
       <robotNamespace>/</robotNamespace>
-    </plugin-->
+    </plugin>
     <!-- Publish joint states so rviz can visualize them. -->
-    <plugin name="joint_state_publisher" filename="libgazebo_ros_joint_state_publisher.so">
+    <!--plugin name="joint_state_publisher" filename="libgazebo_ros_joint_state_publisher.so">
       <jointName>j_shou_yaw, j_shou_pitch, j_prox_pitch, j_dist_pitch,
        j_hand_yaw, j_scoop_yaw, j_ant_pan, j_ant_tilt</jointName>
       <updateRate>10</updateRate>
-    </plugin>
+    </plugin-->
   </gazebo>
 </robot>
