Commit message: Mounted camera on back of antenna panel.

File: ow_lander/urdf/lander.xacro (robot description, xacro)
@@ -1,10 +1,7 @@
 <robot xmlns:xacro="http://ros.org/wiki/xacro" name="lander">
-  <xacro:include filename="$(find ow_lander)/urdf/stereo_mast-triggered.xacro" />
-  <xacro:stereo_mast stereo_mast_parent_link="base_link"
-                     mast_height="1.2"
-                     hfov="70"
-                     img_w="2048" img_h="2048"
-                     update_rate="1"
-                     off_x="-0.2" off_y="0.2" off_z="0.5" />
+  <xacro:include filename="$(find ow_lander)/urdf/stereo_camera_triggered.xacro" />
+  <xacro:stereo_mast stereo_camera_parent_link="l_ant_panel"
+                     hfov="70" img_w="1024" img_h="1024" update_rate="1"
+                     off_x="0.55" off_y="0.05" off_z="0.0" off_R="${pi/2.0}" off_P="${pi}" off_Y="${pi/2.0}" />
   <link
     name="base_link">

File: ow_lander/urdf/stereo_camera_triggered.xacro (robot description, xacro)
@@ -1,12 +1,4 @@
 <?xml version="1.0"?>
 <robot xmlns:xacro="http://ros.org/wiki/xacro" name="stereo_test_mast">
-  <xacro:property name="mast_mass" value="0.1" />
-  <xacro:property name="mast_width" value="0.05" />
-  <xacro:property name="pan_h" value="0.05" />
-  <xacro:property name="pan_h_2" value="0.025" />
-  <xacro:property name="pan_mass" value="0.1" />
-  <xacro:property name="tilt_h" value="0.05" />
-  <xacro:property name="tilt_w" value="0.08" />
-  <xacro:property name="tilt_mass" value="0.1" />
   <xacro:property name="Camera01Name"       value="NavCamStereo" />
   <xacro:property name="Camera01UpdateRate" value="5" />
@@ -14,140 +6,5 @@
   <xacro:property name="camera_head_mass"   value="0.10" />
   <xacro:property name="deg_to_rad"         value="0.0174533" />
-  <!--xacro:include filename="$(find krex2_description)/urdf/nav_lights.xacro" /-->
-  <xacro:macro name="stereo_mast" params="stereo_mast_parent_link mast_height hfov img_w img_h update_rate off_x off_y off_z">
-  <link name="${Camera01Name}_mast_link">
-    <collision>
-      <origin rpy="0 0 0" xyz="0 0 ${mast_height/2}"/>
-      <geometry>
-        <box size="${mast_width} ${mast_width} ${mast_height}"/>
-      </geometry>
-    </collision>
-    <visual>
-      <origin rpy="0 0 0" xyz="0 0 ${mast_height/2}"/>
-      <geometry>
-        <box size="${mast_width} ${mast_width} ${mast_height}"/>
-      </geometry>
-      <material name="Grey"/>
-    </visual>
-    <inertial>
-      <origin rpy="0 0 0" xyz="0 0 ${mast_height/2}"/>
-      <mass value="${mast_mass}"/>
-      <!-- inertia ixx="0.01" ixy="0.0" ixz="0.0" iyy="0.01" iyz="0.0" izz="0.01"/ -->
-      <inertia
-          ixx="${mast_mass / 12.0 * (mast_width*mast_width + mast_height*mast_height)}" ixy="0.0" ixz="0.0"
-          iyy="${mast_mass / 12.0 * (mast_height*mast_height + mast_width*mast_width)}" iyz="0.0"
-          izz="${mast_mass / 12.0 * (mast_width*mast_width + mast_width*mast_width)}"/>
-    </inertial>
-  </link>
-  <gazebo reference="${Camera01Name}_mast_link">
-    <material>Gazebo/Grey</material>
-  </gazebo>
-  <joint name="${Camera01Name}_mast_joint" type="fixed">
-    <parent link="${stereo_mast_parent_link}"/>
-    <child link="${Camera01Name}_mast_link"/>
-    <origin xyz="${off_x} ${off_y} ${off_z}" rpy="0 0 0" />
-  </joint>
-  <link name="${Camera01Name}_pan_link">
-    <collision>
-      <origin rpy="0 0 0" xyz="0 0 ${pan_h_2}"/>
-      <geometry>
-        <box size="0.1 0.1 ${pan_h}"/>
-      </geometry>
-    </collision>
-    <visual>
-      <origin rpy="0 0 0" xyz="0 0 ${pan_h_2}"/>
-      <geometry>
-        <box size="0.1 0.1 ${pan_h}"/>
-      </geometry>
-      <material name="Grey"/>
-    </visual>
-    <inertial>
-      <origin rpy="0 0 0" xyz="0 0 ${pan_h_2}"/>
-      <mass value="${pan_mass}"/>
-      <!-- inertia ixx="0.1" ixy="0.0" ixz="0.0" iyy="0.1" iyz="0.0" izz="0.1"/ -->
-      <inertia
-          ixx="${pan_mass / 12.0 * (0.1*0.1 + pan_h*pan_h)}" ixy="0.0" ixz="0.0"
-          iyy="${pan_mass / 12.0 * (pan_h*pan_h + 0.1*0.1)}" iyz="0.0"
-          izz="${pan_mass / 12.0 * (0.1*0.1 + 0.1*0.1)}"/>
-    </inertial>
-  </link>
-  <gazebo reference="${Camera01Name}_pan_link">
-    <material>Gazebo/Grey</material>
-  </gazebo>
-  <joint name="${Camera01Name}_pan_joint" type="revolute">
-    <parent link="${Camera01Name}_mast_link"/>
-    <child link="${Camera01Name}_pan_link"/>
-    <origin xyz="0 0 ${mast_height}" rpy="0 0 0" />
-    <axis xyz="0 0 1"/>
-    <limit lower="${-1.0 * pi}" upper="${1.0 * pi}" effort="-1" velocity="-1"/>
-  </joint>
-  <transmission name="pan_transmission">
-    <type>transmission_interface/SimpleTransmission</type>
-    <joint name="${Camera01Name}_pan_joint">
-      <hardwareInterface>hardware_interface/EffortJointInterface</hardwareInterface>
-    </joint>
-    <actuator name="pan_motor">
-      <mechanicalReduction>1</mechanicalReduction>
-    </actuator>
-  </transmission>
-  <link name="${Camera01Name}_tilt_link">
-    <collision>
-      <origin rpy="0 0 0" xyz="0 0 ${tilt_h/2}"/>
-      <geometry>
-        <box size="${tilt_w} ${tilt_w} ${tilt_h}"/>
-      </geometry>
-    </collision>
-    <visual>
-      <origin rpy="0 0 0" xyz="0 0 ${tilt_h/2}"/>
-      <geometry>
-        <box size="${tilt_w} ${tilt_w} ${tilt_h}"/>
-      </geometry>
-      <material name="Grey"/>
-    </visual>
-    <inertial>
-      <origin rpy="0 0 0" xyz="0 0 ${tilt_h/2}"/>
-      <mass value="${tilt_mass}"/>
-      <!-- inertia ixx="0.1" ixy="0.0" ixz="0.0" iyy="0.1" iyz="0.0" izz="0.1"/ -->
-      <!-- see https://github.com/ros-simulation/gazebo_ros_demos/blob/master/rrbot_description/urdf/rrbot.xacro for box formula -->
-      <!-- https://en.wikipedia.org/wiki/List_of_moments_of_inertia -->
-      <!-- inertia
-          ixx="${mass / 12.0 * (depth*depth + height*height)}" ixy="0.0" ixz="0.0"
-          iyy="${mass / 12.0 * (height*height + width*width)}" iyz="0.0"
-          izz="${mass / 12.0 * (depth*depth + width*width)}"/ -->
-     <inertia
-          ixx="${tilt_mass / 12.0 * (tilt_w*tilt_w + tilt_h*tilt_h)}" ixy="0.0" ixz="0.0"
-          iyy="${tilt_mass / 12.0 * (tilt_h*tilt_h + tilt_w*tilt_w)}" iyz="0.0"
-          izz="${tilt_mass / 12.0 * (tilt_w*tilt_w + tilt_w*tilt_w)}"/>
-    </inertial>
-  </link>
-  <!-- ==== nav_lights on fixed joint ================================= -->
-  <!-- NOTE: preserveFixedJoint tag REQUIRED for URDF to SDF conversion -->
-  <!--xacro:nav_lights />
-  <joint name="nav_lights_joint" type="fixed">
-    <parent link="${Camera01Name}_tilt_link"/>
-    <child link="nav_lights_link"/>
-    <origin xyz="0.0 0.0 0.3" rpy="0.0 0.0 0.0" />
-    <axis xyz="0 1 0"/>
-  </joint>
-  <gazebo reference='nav_lights_joint'>
-    <preserveFixedJoint>true</preserveFixedJoint>
-  </gazebo-->
-  <joint name="${Camera01Name}_tilt_joint" type="revolute">
-    <parent link="${Camera01Name}_pan_link"/>
-    <child link="${Camera01Name}_tilt_link"/>
-    <origin xyz="0 0 ${pan_h}" rpy="0 0.2 0" />
-    <axis xyz="0 1 0"/>
-    <!-- setting limits to -1 should make them unbounded in Gazebo and force use of ros_control limits -->
-    <limit lower="-0.9" upper="1.0" effort="-1" velocity="-1"/>
-  </joint>
-  <transmission name="tilt_transmission">
-    <type>transmission_interface/SimpleTransmission</type>
-    <joint name="${Camera01Name}_tilt_joint">
-      <hardwareInterface>hardware_interface/EffortJointInterface</hardwareInterface>
-    </joint>
-    <actuator name="tilt_motor">
-      <mechanicalReduction>1</mechanicalReduction>
-    </actuator>
-  </transmission>
+  <xacro:macro name="stereo_mast" params="stereo_camera_parent_link hfov img_w img_h update_rate off_x off_y off_z off_R off_P off_Y">
   <link name="${Camera01Name}_head_link">
     <collision>
@@ -188,4 +45,9 @@
    </inertial>
   </link>
+  <joint name="${Camera01Name}_joint" type="fixed">
+    <parent link="${stereo_camera_parent_link}"/>
+    <child link="${Camera01Name}_head_link"/>
+    <origin xyz="${off_x} ${off_y} ${off_z}" rpy="${off_R} ${off_P} ${off_Y}" />
+  </joint>
   <!-- example for stereo setup is here: -->
   <!-- https://bitbucket.org/osrf/drcsim/src/52a691b8956045442ef22ba0aaee4520716807ff/multisense_sl_description/urdf/multisense_sl.urdf?at=default#cl-200 -->
@@ -200,5 +62,5 @@
   </joint>
   <joint name="leftCamera_optical_joint" type="fixed">
-    <origin xyz="0.0 0.0 0.0" rpy="-${pi/2.0} 0 -${pi/2.0}"/>
+    <origin xyz="0.0 0.0 0.0" rpy="0 0 0"/>
     <parent link="${Camera01Name}Left_link"/>
     <child link="${Camera01Name}Left_optical_frame"/>
@@ -213,5 +75,5 @@
   </joint>
   <joint name="rightCamera_optical_joint" type="fixed">
-    <origin xyz="0.0 0.0 0.0" rpy="-${pi/2.0} 0 -${pi/2.0}"/>
+    <origin xyz="0.0 0.0 0.0" rpy="0 0 0"/>
     <parent link="${Camera01Name}Right_link"/>
     <child link="${Camera01Name}Right_optical_frame"/>
@@ -271,10 +133,10 @@
   <link name="${Camera01Name}Center_optical_frame"/>
   <joint name="CenterCamera_joint" type="fixed">
-    <origin xyz="0.025 0.0 0.0" rpy="0 0 0"/>
+    <origin xyz="0.0 0.0 0.0" rpy="0 0 0"/>
     <parent link="${Camera01Name}_head_link"/>
     <child link="${Camera01Name}Center_link"/>
   </joint>
   <joint name="CenterCamera_optical_joint" type="fixed">
-    <origin xyz="0.0 0.0 0.0" rpy="-${pi/2.0} 0 -${pi/2.0}"/>
+    <origin xyz="0.0 0.0 0.0" rpy="0 0 0"/>
     <parent link="${Camera01Name}Center_link"/>
     <child link="${Camera01Name}Center_optical_frame"/>
@@ -315,11 +177,4 @@
     </sensor>
   </gazebo>
-  <!-- Camera Joint -->
-  <joint name="${Camera01Name}_camera_joint" type="fixed">
-    <axis xyz="0 1 0" />
-    <origin xyz="0.005 0 ${tilt_h}" rpy="0 0 0"/>
-    <parent link="${Camera01Name}_tilt_link"/>
-    <child link="${Camera01Name}_head_link"/>
-  </joint>
   </xacro:macro>
 </robot>

Commit message: Use primitives instead of lander body for collision to speed up physics and Gazebo real-time factor. Set velocity limit on joints.

File: ow_lander/urdf/lander.xacro (robot description, xacro)
@@ -35,4 +35,28 @@
     </visual>
     <collision>
+      <origin xyz="1.064 1.064 -0.05" rpy="0 0 0" />
+      <geometry>
+        <sphere radius="0.125" />
+      </geometry>
+    </collision>
+    <collision>
+      <origin xyz="-1.064 1.064 -0.05" rpy="0 0 0" />
+      <geometry>
+        <sphere radius="0.125" />
+      </geometry>
+    </collision>
+    <collision>
+      <origin xyz="1.064 -1.064 -0.05" rpy="0 0 0" />
+      <geometry>
+        <sphere radius="0.125" />
+      </geometry>
+    </collision>
+    <collision>
+      <origin xyz="-1.064 -1.064 -0.05" rpy="0 0 0" />
+      <geometry>
+        <sphere radius="0.125" />
+      </geometry>
+    </collision>
+    <!--collision>
       <origin
         xyz="0 0 0"
@@ -42,5 +66,5 @@
           filename="package://ow_lander/meshes/base_link.STL" />
       </geometry>
-    </collision>
+    </collision-->
   </link>
   <link
@@ -97,4 +121,5 @@
       xyz="0 0 -1" />
     <dynamics damping="50" />
+    <limit effort="1000.0" velocity="0.2" />
   </joint>
   <transmission name="shou_yaw_transmission">
@@ -160,4 +185,5 @@
       xyz="0 0 -1" />
     <dynamics damping="50" />
+    <limit effort="1000.0" velocity="0.2" />
   </joint>
   <transmission name="shou_pitch_transmission">
@@ -223,4 +249,5 @@
       xyz="0 0 -1" />
     <dynamics damping="50" />
+    <limit effort="1000.0" velocity="0.2" />
   </joint>
   <transmission name="prox_pitch_transmission">
@@ -286,4 +313,5 @@
       xyz="0 0 1" />
     <dynamics damping="50" />
+    <limit effort="1000.0" velocity="0.2" />
   </joint>
   <transmission name="dist_pitch_transmission">
@@ -349,4 +377,5 @@
       xyz="0 0 -1" />
     <dynamics damping="50" />
+    <limit effort="1000.0" velocity="0.2" />
   </joint>
   <transmission name="hand_yaw_transmission">
@@ -412,4 +441,5 @@
       xyz="0 0 -1" />
     <dynamics damping="50" />
+    <limit effort="1000.0" velocity="0.2" />
   </joint>
   <transmission name="scoop_yaw_transmission">
@@ -475,4 +505,5 @@
       xyz="0 0 -1" />
     <dynamics damping="50" />
+    <limit effort="1000.0" velocity="0.2" />
   </joint>
   <transmission name="ant_pan_transmission">
@@ -538,4 +569,5 @@
       xyz="0 0 -1" />
     <dynamics damping="50" />
+    <limit effort="1000.0" velocity="0.2" />
   </joint>
   <transmission name="ant_tilt_transmission">

Commit message: Cleaned up /launch and /config, use lander.xacro for planning (not lander_urdf_v9 anymore). Save trajectories in ~/.ros/ and removes bag and csv.

File: ow_lander/urdf/lander.xacro (robot description, xacro)
@@ -185,5 +185,5 @@
       xyz="0 0 -1" />
     <dynamics damping="50" />
-    <limit effort="1000.0" velocity="0.2" />
+    <limit effort="1000.0" velocity="0.2" lower="-0.05" upper="2.2"/>
   </joint>
   <transmission name="shou_pitch_transmission">

Commit message: Cleaned up scripts and names, shou pitch to revolute, verified depth

File: ow_lander/urdf/lander.xacro (robot description, xacro)
@@ -121,5 +121,5 @@
       xyz="0 0 -1" />
     <dynamics damping="50" />
-    <limit effort="1000.0" velocity="0.2" />
+    <limit effort="1000.0" velocity="0.2"/>
   </joint>
   <transmission name="shou_yaw_transmission">
@@ -174,5 +174,5 @@
   <joint
     name="j_shou_pitch"
-    type="continuous">
+    type="revolute">
     <origin
       xyz="0.16 0 0"
@@ -185,5 +185,5 @@
       xyz="0 0 -1" />
     <dynamics damping="50" />
-    <limit effort="1000.0" velocity="0.2" lower="-0.05" upper="2.2"/>
+    <limit effort="1000.0" velocity="0.2" lower="0.05" upper="2.2"/>
   </joint>
   <transmission name="shou_pitch_transmission">
@@ -267,5 +267,5 @@
         rpy="0 0 0" />
       <mass
-        value="4.24254588886639" />
+        value="1.24254588886639" />
       <inertia
         ixx="0.00600454075116932"
@@ -331,5 +331,5 @@
         rpy="0 0 0" />
       <mass
-        value="3.08554586923443" />
+        value="1.08554586923443" />
       <inertia
         ixx="0.00868815536634117"

Commit message: Removed /ros/ros.h, tuned controllers and masses

File: ow_lander/urdf/lander.xacro (robot description, xacro)
@@ -110,5 +110,5 @@
   <joint
     name="j_shou_yaw"
-    type="continuous">
+    type="revolute">
     <origin
       xyz="0.79 0.175 0.27"
@@ -121,5 +121,5 @@
       xyz="0 0 -1" />
     <dynamics damping="50" />
-    <limit effort="1000.0" velocity="0.2"/>
+    <limit effort="1000.0" velocity="0.2" lower="-1.5" upper="1.5"/>
   </joint>
   <transmission name="shou_yaw_transmission">
@@ -174,5 +174,5 @@
   <joint
     name="j_shou_pitch"
-    type="revolute">
+    type="continuous">
     <origin
       xyz="0.16 0 0"
@@ -267,5 +267,5 @@
         rpy="0 0 0" />
       <mass
-        value="1.24254588886639" />
+        value="4.24254588886639" />
       <inertia
         ixx="0.00600454075116932"
@@ -331,5 +331,5 @@
         rpy="0 0 0" />
       <mass
-        value="1.08554586923443" />
+        value="3.08554586923443" />
       <inertia
         ixx="0.00868815536634117"

Commit message: Clean up post code review. Removed joint_limits.yaml. Added pkg level readme. Deleted more launch files

File: ow_lander/urdf/lander.xacro (robot description, xacro)
@@ -121,5 +121,5 @@
       xyz="0 0 -1" />
     <dynamics damping="50" />
-    <limit effort="1000.0" velocity="0.2" lower="-1.5" upper="1.5"/>
+    <limit effort="1000.0" velocity="0.5" lower="-1.5" upper="1.5"/>
   </joint>
   <transmission name="shou_yaw_transmission">
@@ -185,5 +185,5 @@
       xyz="0 0 -1" />
     <dynamics damping="50" />
-    <limit effort="1000.0" velocity="0.2" lower="0.05" upper="2.2"/>
+    <limit effort="1000.0" velocity="0.5" lower="0.05" upper="2.2"/>
   </joint>
   <transmission name="shou_pitch_transmission">
@@ -249,5 +249,5 @@
       xyz="0 0 -1" />
     <dynamics damping="50" />
-    <limit effort="1000.0" velocity="0.2" />
+    <limit effort="1000.0" velocity="0.5" />
   </joint>
   <transmission name="prox_pitch_transmission">
@@ -313,5 +313,5 @@
       xyz="0 0 1" />
     <dynamics damping="50" />
-    <limit effort="1000.0" velocity="0.2" />
+    <limit effort="1000.0" velocity="0.5" />
   </joint>
   <transmission name="dist_pitch_transmission">
@@ -377,5 +377,5 @@
       xyz="0 0 -1" />
     <dynamics damping="50" />
-    <limit effort="1000.0" velocity="0.2" />
+    <limit effort="1000.0" velocity="0.5" />
   </joint>
   <transmission name="hand_yaw_transmission">
@@ -441,5 +441,5 @@
       xyz="0 0 -1" />
     <dynamics damping="50" />
-    <limit effort="1000.0" velocity="0.2" />
+    <limit effort="1000.0" velocity="0.5" />
   </joint>
   <transmission name="scoop_yaw_transmission">
@@ -505,5 +505,5 @@
       xyz="0 0 -1" />
     <dynamics damping="50" />
-    <limit effort="1000.0" velocity="0.2" />
+    <limit effort="1000.0" velocity="0.5" />
   </joint>
   <transmission name="ant_pan_transmission">
@@ -569,5 +569,5 @@
       xyz="0 0 -1" />
     <dynamics damping="50" />
-    <limit effort="1000.0" velocity="0.2" />
+    <limit effort="1000.0" velocity="0.5" />
   </joint>
   <transmission name="ant_tilt_transmission">

Commit message: Turned on self-collisions between lander parts. Added freeze_base_link capability. Disabled collisions between base_link and terrain when base_link is frozen.

File: ow_lander/urdf/lander.xacro (robot description, xacro)
@@ -4,6 +4,14 @@
                      hfov="70" img_w="1024" img_h="1024" update_rate="1"
                      off_x="0.55" off_y="0.05" off_z="0.0" off_R="${pi/2.0}" off_P="${pi}" off_Y="${pi/2.0}" />
-  <link
-    name="base_link">
+  <xacro:arg name="freeze_base_link" default="false"/>
+  <xacro:if value="$(arg freeze_base_link)">
+    <!-- Rigidly fix robot to world: http://gazebosim.org/tutorials/?tut=ros_urdf#RigidlyFixingAModeltotheWorld -->
+    <link name="world"/>
+    <joint name="fixed" type="fixed">
+      <parent link="world"/>
+      <child link="base_link"/>
+    </joint>
+  </xacro:if>
+  <link name="base_link">
     <inertial>
       <origin
@@ -35,28 +43,4 @@
     </visual>
     <collision>
-      <origin xyz="1.064 1.064 -0.05" rpy="0 0 0" />
-      <geometry>
-        <sphere radius="0.125" />
-      </geometry>
-    </collision>
-    <collision>
-      <origin xyz="-1.064 1.064 -0.05" rpy="0 0 0" />
-      <geometry>
-        <sphere radius="0.125" />
-      </geometry>
-    </collision>
-    <collision>
-      <origin xyz="1.064 -1.064 -0.05" rpy="0 0 0" />
-      <geometry>
-        <sphere radius="0.125" />
-      </geometry>
-    </collision>
-    <collision>
-      <origin xyz="-1.064 -1.064 -0.05" rpy="0 0 0" />
-      <geometry>
-        <sphere radius="0.125" />
-      </geometry>
-    </collision>
-    <!--collision>
       <origin
         xyz="0 0 0"
@@ -66,8 +50,22 @@
           filename="package://ow_lander/meshes/base_link.STL" />
       </geometry>
-    </collision-->
-  </link>
-  <link
-    name="l_shou">
+    </collision>
+  </link>
+  <gazebo reference="base_link">
+    <selfCollide>1</selfCollide>
+    <!-- If freezing the lander in place, turn off collisions with the terrain
+         because these collisions cause strange physics side effects. For this
+         to work, the terrain must use a different collide_bitmask. -->
+    <xacro:if value="$(arg freeze_base_link)">
+      <collision>
+        <surface>
+          <contact>
+            <collide_bitmask>0x0001</collide_bitmask>
+          </contact>
+        </surface>
+      </collision>
+    </xacro:if>
+  </gazebo>
+  <link name="l_shou">
     <inertial>
       <origin
@@ -108,4 +106,7 @@
     </collision>
   </link>
+  <gazebo reference="l_shou">
+    <selfCollide>1</selfCollide>
+  </gazebo>
   <joint
     name="j_shou_yaw"
@@ -132,6 +133,5 @@
     </actuator>
   </transmission>
-  <link
-    name="l_prox">
+  <link name="l_prox">
     <inertial>
       <origin
@@ -172,4 +172,7 @@
     </collision>
   </link>
+  <gazebo reference="l_prox">
+    <selfCollide>1</selfCollide>
+  </gazebo>
   <joint
     name="j_shou_pitch"
@@ -196,6 +199,5 @@
     </actuator>
   </transmission>
-  <link
-    name="l_dist">
+  <link name="l_dist">
     <inertial>
       <origin
@@ -236,4 +238,7 @@
     </collision>
   </link>
+  <gazebo reference="l_dist">
+    <selfCollide>1</selfCollide>
+  </gazebo>
   <joint
     name="j_prox_pitch"
@@ -260,6 +265,5 @@
     </actuator>
   </transmission>
-  <link
-    name="l_wrist">
+  <link name="l_wrist">
     <inertial>
       <origin
@@ -300,4 +304,7 @@
     </collision>
   </link>
+  <gazebo reference="l_wrist">
+    <selfCollide>1</selfCollide>
+  </gazebo>
   <joint
     name="j_dist_pitch"
@@ -324,6 +331,5 @@
     </actuator>
   </transmission>
-  <link
-    name="l_hand">
+  <link name="l_hand">
     <inertial>
       <origin
@@ -364,4 +370,7 @@
     </collision>
   </link>
+  <gazebo reference="l_hand">
+    <selfCollide>1</selfCollide>
+  </gazebo>
   <joint
     name="j_hand_yaw"
@@ -388,6 +397,5 @@
     </actuator>
   </transmission>
-  <link
-    name="l_scoop">
+  <link name="l_scoop">
     <inertial>
       <origin
@@ -428,4 +436,7 @@
     </collision>
   </link>
+  <gazebo reference="l_scoop">
+    <selfCollide>1</selfCollide>
+  </gazebo>
   <joint
     name="j_scoop_yaw"
@@ -452,6 +463,5 @@
     </actuator>
   </transmission>
-  <link
-    name="l_ant_foot">
+  <link name="l_ant_foot">
     <inertial>
       <origin
@@ -492,4 +502,7 @@
     </collision>
   </link>
+  <gazebo reference="l_ant_foot">
+    <selfCollide>1</selfCollide>
+  </gazebo>
   <joint
     name="j_ant_pan"
@@ -516,6 +529,5 @@
     </actuator>
   </transmission>
-  <link
-    name="l_ant_panel">
+  <link name="l_ant_panel">
     <inertial>
       <origin
@@ -556,4 +568,7 @@
     </collision>
   </link>
+  <gazebo reference="l_ant_panel">
+    <selfCollide>1</selfCollide>
+  </gazebo>
   <joint
     name="j_ant_tilt"

Commit message: Disable scoop collision with terrain.

File: ow_lander/urdf/lander.xacro (robot description, xacro)
@@ -438,4 +438,13 @@
   <gazebo reference="l_scoop">
     <selfCollide>1</selfCollide>
+    <!-- Turn off collisions with the terrain so scoop can go underground. For
+         this to work, the terrain must use a different collide_bitmask. -->
+    <collision>
+      <surface>
+        <contact>
+          <collide_bitmask>0x0002</collide_bitmask>
+        </contact>
+      </surface>
+    </collision>
   </gazebo>
   <joint
