Commit message: Tuned parameters, added initial pose in spawn.launch

File: ow_lander/urdf/lander.xacro (robot description, xacro)
@@ -122,5 +122,5 @@
       xyz="0 0 -1" />
     <dynamics damping="50" />
-    <limit effort="1000.0" velocity="0.5" lower="-1.5" upper="1.5"/>
+    <limit effort="1000.0" velocity="0.4" lower="-1.5" upper="1.5"/>
   </joint>
   <transmission name="shou_yaw_transmission">
@@ -188,5 +188,5 @@
       xyz="0 0 -1" />
     <dynamics damping="50" />
-    <limit effort="1000.0" velocity="0.5" lower="0.05" upper="2.2"/>
+    <limit effort="1000.0" velocity="0.4" lower="0.05" upper="2.2"/>
   </joint>
   <transmission name="shou_pitch_transmission">
@@ -205,5 +205,5 @@
         rpy="0 0 0" />
       <mass
-        value="7.47049693100743" />
+        value="3.47049693100743" />
       <inertia
         ixx="0.00621200133375043"
@@ -254,5 +254,5 @@
       xyz="0 0 -1" />
     <dynamics damping="50" />
-    <limit effort="1000.0" velocity="0.5" />
+    <limit effort="1000.0" velocity="0.4" />
   </joint>
   <transmission name="prox_pitch_transmission">
@@ -271,5 +271,5 @@
         rpy="0 0 0" />
       <mass
-        value="4.24254588886639" />
+        value="1.24254588886639" />
       <inertia
         ixx="0.00600454075116932"
@@ -320,5 +320,5 @@
       xyz="0 0 1" />
     <dynamics damping="50" />
-    <limit effort="1000.0" velocity="0.5" />
+    <limit effort="1000.0" velocity="0.4" />
   </joint>
   <transmission name="dist_pitch_transmission">
@@ -337,5 +337,5 @@
         rpy="0 0 0" />
       <mass
-        value="3.08554586923443" />
+        value="1.08554586923443" />
       <inertia
         ixx="0.00868815536634117"
@@ -395,5 +395,5 @@
       xyz="0 0 -1" />
     <dynamics damping="50" />
-    <limit effort="1000.0" velocity="0.5" />
+    <limit effort="1000.0" velocity="0.4" />
   </joint>
   <transmission name="hand_yaw_transmission">
@@ -470,5 +470,5 @@
       xyz="0 0 -1" />
     <dynamics damping="50" />
-    <limit effort="1000.0" velocity="0.5" />
+    <limit effort="1000.0" velocity="0.4" />
   </joint>
   <transmission name="scoop_yaw_transmission">
@@ -536,5 +536,5 @@
       xyz="0 0 -1" />
     <dynamics damping="50" />
-    <limit effort="1000.0" velocity="0.5" />
+    <limit effort="1000.0" velocity="0.4" />
   </joint>
   <transmission name="ant_pan_transmission">
@@ -602,5 +602,5 @@
       xyz="0 0 -1" />
     <dynamics damping="50" />
-    <limit effort="1000.0" velocity="0.5" />
+    <limit effort="1000.0" velocity="0.4" />
   </joint>
   <transmission name="ant_tilt_transmission">

Commit message: Added headers, initial position commander, cleaner trajectory

File: ow_lander/urdf/lander.xacro (robot description, xacro)
@@ -122,5 +122,5 @@
       xyz="0 0 -1" />
     <dynamics damping="50" />
-    <limit effort="1000.0" velocity="0.4" lower="-1.5" upper="1.5"/>
+    <limit effort="1000.0" velocity="0.4" lower="-1.8" upper="1.8"/>
   </joint>
   <transmission name="shou_yaw_transmission">

Commit message: Added lights to lander's xacro description.

File: ow_lander/urdf/lander.xacro (robot description, xacro)
@@ -1,7 +1,10 @@
 <robot xmlns:xacro="http://ros.org/wiki/xacro" name="lander">
   <xacro:include filename="$(find ow_lander)/urdf/stereo_camera_triggered.xacro" />
-  <xacro:stereo_mast stereo_camera_parent_link="l_ant_panel"
+  <xacro:stereo_camera stereo_camera_parent_link="l_ant_panel"
                      hfov="70" img_w="1024" img_h="1024" update_rate="1"
                      off_x="0.55" off_y="0.05" off_z="0.0" off_R="${pi/2.0}" off_P="${pi}" off_Y="${pi/2.0}" />
+  <xacro:include filename="$(find ow_lander)/urdf/lander_lights.xacro" />
+  <xacro:lander_lights lander_lights_parent_link="l_ant_panel"
+                     off_x="0.85" off_y="0.07" off_z="0.0" off_R="-${pi/2.0}" off_P="0.0" off_Y="0.0" />
   <xacro:arg name="freeze_base_link" default="false"/>
   <xacro:if value="$(arg freeze_base_link)">

File: ow_lander/urdf/stereo_camera_triggered.xacro (robot description, xacro)
@@ -1,4 +1,4 @@
 <?xml version="1.0"?>
-<robot xmlns:xacro="http://ros.org/wiki/xacro" name="stereo_test_mast">
+<robot xmlns:xacro="http://ros.org/wiki/xacro" name="stereo_camera">
   <xacro:property name="Camera01Name"       value="NavCamStereo" />
   <xacro:property name="Camera01UpdateRate" value="5" />
@@ -6,5 +6,5 @@
   <xacro:property name="camera_head_mass"   value="0.10" />
   <xacro:property name="deg_to_rad"         value="0.0174533" />
-  <xacro:macro name="stereo_mast" params="stereo_camera_parent_link hfov img_w img_h update_rate off_x off_y off_z off_R off_P off_Y">
+  <xacro:macro name="stereo_camera" params="stereo_camera_parent_link hfov img_w img_h update_rate off_x off_y off_z off_R off_P off_Y">
   <link name="${Camera01Name}_head_link">
     <collision>

Commit message: Set reasonable exposure and energy_conversion params on lander cameras. Added shaders to lander so it can be properly lit by scene's sunIntensity values.

File: ow_lander/urdf/lander.xacro (robot description, xacro)
@@ -56,4 +56,14 @@
   </link>
   <gazebo reference="base_link">
+    <visual>
+      <material>
+        <diffuse>0.792 0.819 0.933 1</diffuse>
+        <specular>0.4 0.4 0.4 1</specular>
+        <script>
+          <uri>package://ow_lander/materials/scripts</uri>
+          <name>ow/lander</name>
+        </script>
+      </material>
+    </visual>
     <selfCollide>1</selfCollide>
     <!-- If freezing the lander in place, turn off collisions with the terrain
@@ -110,4 +120,14 @@
   </link>
   <gazebo reference="l_shou">
+    <visual>
+      <material>
+        <diffuse>0.898 0.917 0.929 1</diffuse>
+        <specular>0.4 0.4 0.4 1</specular>
+        <script>
+          <uri>package://ow_lander/materials/scripts</uri>
+          <name>ow/lander</name>
+        </script>
+      </material>
+    </visual>
     <selfCollide>1</selfCollide>
   </gazebo>
@@ -176,4 +196,14 @@
   </link>
   <gazebo reference="l_prox">
+    <visual>
+      <material>
+        <diffuse>0.898 0.917 0.929 1</diffuse>
+        <specular>0.4 0.4 0.4 1</specular>
+        <script>
+          <uri>package://ow_lander/materials/scripts</uri>
+          <name>ow/lander</name>
+        </script>
+      </material>
+    </visual>
     <selfCollide>1</selfCollide>
   </gazebo>
@@ -242,4 +272,14 @@
   </link>
   <gazebo reference="l_dist">
+    <visual>
+      <material>
+        <diffuse>0.898 0.917 0.929 1</diffuse>
+        <specular>0.4 0.4 0.4 1</specular>
+        <script>
+          <uri>package://ow_lander/materials/scripts</uri>
+          <name>ow/lander</name>
+        </script>
+      </material>
+    </visual>
     <selfCollide>1</selfCollide>
   </gazebo>
@@ -308,4 +348,14 @@
   </link>
   <gazebo reference="l_wrist">
+    <visual>
+      <material>
+        <diffuse>0.898 0.917 0.929 1</diffuse>
+        <specular>0.4 0.4 0.4 1</specular>
+        <script>
+          <uri>package://ow_lander/materials/scripts</uri>
+          <name>ow/lander</name>
+        </script>
+      </material>
+    </visual>
     <selfCollide>1</selfCollide>
   </gazebo>
@@ -374,4 +424,14 @@
   </link>
   <gazebo reference="l_hand">
+    <visual>
+      <material>
+        <diffuse>0.898 0.917 0.929 1</diffuse>
+        <specular>0.4 0.4 0.4 1</specular>
+        <script>
+          <uri>package://ow_lander/materials/scripts</uri>
+          <name>ow/lander</name>
+        </script>
+      </material>
+    </visual>
     <selfCollide>1</selfCollide>
     <!-- Turn off collisions with the terrain so scoop can go underground. For
@@ -449,4 +509,14 @@
   </link>
   <gazebo reference="l_scoop">
+    <visual>
+      <material>
+        <diffuse>0.898 0.917 0.929 1</diffuse>
+        <specular>0.4 0.4 0.4 1</specular>
+        <script>
+          <uri>package://ow_lander/materials/scripts</uri>
+          <name>ow/lander</name>
+        </script>
+      </material>
+    </visual>
     <selfCollide>1</selfCollide>
     <!-- Turn off collisions with the terrain so scoop can go underground. For
@@ -524,4 +594,14 @@
   </link>
   <gazebo reference="l_ant_foot">
+    <visual>
+      <material>
+        <diffuse>0.294 0.294 0.294 1</diffuse>
+        <specular>0.4 0.4 0.4 1</specular>
+        <script>
+          <uri>package://ow_lander/materials/scripts</uri>
+          <name>ow/lander</name>
+        </script>
+      </material>
+    </visual>
     <selfCollide>1</selfCollide>
   </gazebo>
@@ -590,4 +670,14 @@
   </link>
   <gazebo reference="l_ant_panel">
+    <visual>
+      <material>
+        <diffuse>0.294 0.294 0.294 1</diffuse>
+        <specular>0.4 0.4 0.4 1</specular>
+        <script>
+          <uri>package://ow_lander/materials/scripts</uri>
+          <name>ow/lander</name>
+        </script>
+      </material>
+    </visual>
     <selfCollide>1</selfCollide>
   </gazebo>

File: ow_lander/urdf/stereo_camera_triggered.xacro (robot description, xacro)
@@ -126,6 +126,6 @@
       <plugin name="LensFlare" filename="libLensFlareSensorPlugin.so"/>
       <plugin name="CameraSim" filename="libIRGCameraSimSensorPlugin.so" >
-        <exposure>1.0</exposure>
-        <gain>1.0</gain>
+        <exposure>0.033333</exposure>
+        <energy_conversion>0.0075</energy_conversion>
       </plugin>
     </sensor>

Commit message: Model simulated camera after Mastcam-34 properties.

File: ow_lander/urdf/lander.xacro (robot description, xacro)
@@ -2,5 +2,5 @@
   <xacro:include filename="$(find ow_lander)/urdf/stereo_camera_triggered.xacro" />
   <xacro:stereo_camera stereo_camera_parent_link="l_ant_panel"
-                     hfov="70" img_w="1024" img_h="1024" update_rate="1"
+                     hfov="21" img_w="1600" img_h="1200" update_rate="1"
                      off_x="0.55" off_y="0.05" off_z="0.0" off_R="${pi/2.0}" off_P="${pi}" off_Y="${pi/2.0}" />
   <xacro:include filename="$(find ow_lander)/urdf/lander_lights.xacro" />

File: ow_lander/urdf/stereo_camera_triggered.xacro (robot description, xacro)
@@ -3,6 +3,6 @@
   <xacro:property name="Camera01Name"       value="NavCamStereo" />
   <xacro:property name="Camera01UpdateRate" value="5" />
-  <xacro:property name="camera_baseline"    value="0.40" />
-  <xacro:property name="camera_head_mass"   value="0.10" />
+  <xacro:property name="camera_baseline"    value="0.2" />
+  <xacro:property name="camera_head_mass"   value="0.1" />
   <xacro:property name="deg_to_rad"         value="0.0174533" />
   <xacro:macro name="stereo_camera" params="stereo_camera_parent_link hfov img_w img_h update_rate off_x off_y off_z off_R off_P off_Y">

Commit message: Do not render lander into irradiance maps.

File: ow_lander/urdf/lander.xacro (robot description, xacro)
@@ -1,10 +1,14 @@
 <robot xmlns:xacro="http://ros.org/wiki/xacro" name="lander">
+  <!-- A non-standard bitmask to prevent the lander from rendering into the irradiance environment map -->
+  <xacro:property name="vis_mask" value="0x00010000" />
   <xacro:include filename="$(find ow_lander)/urdf/stereo_camera_triggered.xacro" />
   <xacro:stereo_camera stereo_camera_parent_link="l_ant_panel"
                      hfov="21" img_w="1600" img_h="1200" update_rate="1"
-                     off_x="0.55" off_y="0.05" off_z="0.0" off_R="${pi/2.0}" off_P="${pi}" off_Y="${pi/2.0}" />
+                     off_x="0.55" off_y="0.05" off_z="0.0" off_R="${pi/2.0}" off_P="${pi}" off_Y="${pi/2.0}"
+                     vis_mask="${vis_mask}" />
   <xacro:include filename="$(find ow_lander)/urdf/lander_lights.xacro" />
   <xacro:lander_lights lander_lights_parent_link="l_ant_panel"
-                     off_x="0.85" off_y="0.07" off_z="0.0" off_R="-${pi/2.0}" off_P="0.0" off_Y="0.0" />
+                     off_x="0.85" off_y="0.07" off_z="0.0" off_R="-${pi/2.0}" off_P="0.0" off_Y="0.0"
+                     vis_mask="${vis_mask}" />
   <xacro:arg name="freeze_base_link" default="false"/>
   <xacro:if value="$(arg freeze_base_link)">
@@ -65,4 +69,7 @@
         </script>
       </material>
+      <plugin name="visibility" filename="libIRGVisibilityPlugin.so">
+        <visibility_bitmask>${vis_mask}</visibility_bitmask>
+      </plugin>
     </visual>
     <selfCollide>1</selfCollide>
@@ -129,4 +136,7 @@
         </script>
       </material>
+      <plugin name="visibility" filename="libIRGVisibilityPlugin.so">
+        <visibility_bitmask>${vis_mask}</visibility_bitmask>
+      </plugin>
     </visual>
     <selfCollide>1</selfCollide>
@@ -205,4 +215,7 @@
         </script>
       </material>
+      <plugin name="visibility" filename="libIRGVisibilityPlugin.so">
+        <visibility_bitmask>${vis_mask}</visibility_bitmask>
+      </plugin>
     </visual>
     <selfCollide>1</selfCollide>
@@ -281,4 +294,7 @@
         </script>
       </material>
+      <plugin name="visibility" filename="libIRGVisibilityPlugin.so">
+        <visibility_bitmask>${vis_mask}</visibility_bitmask>
+      </plugin>
     </visual>
     <selfCollide>1</selfCollide>
@@ -357,4 +373,7 @@
         </script>
       </material>
+      <plugin name="visibility" filename="libIRGVisibilityPlugin.so">
+        <visibility_bitmask>${vis_mask}</visibility_bitmask>
+      </plugin>
     </visual>
     <selfCollide>1</selfCollide>
@@ -433,4 +452,7 @@
         </script>
       </material>
+      <plugin name="visibility" filename="libIRGVisibilityPlugin.so">
+        <visibility_bitmask>${vis_mask}</visibility_bitmask>
+      </plugin>
     </visual>
     <selfCollide>1</selfCollide>
@@ -519,4 +541,7 @@
         </script>
       </material>
+      <plugin name="visibility" filename="libIRGVisibilityPlugin.so">
+        <visibility_bitmask>${vis_mask}</visibility_bitmask>
+      </plugin>
     </visual>
     <selfCollide>1</selfCollide>
@@ -605,4 +630,7 @@
         </script>
       </material>
+      <plugin name="visibility" filename="libIRGVisibilityPlugin.so">
+        <visibility_bitmask>${vis_mask}</visibility_bitmask>
+      </plugin>
     </visual>
     <selfCollide>1</selfCollide>
@@ -681,4 +709,7 @@
         </script>
       </material>
+      <plugin name="visibility" filename="libIRGVisibilityPlugin.so">
+        <visibility_bitmask>${vis_mask}</visibility_bitmask>
+      </plugin>
     </visual>
     <selfCollide>1</selfCollide>

File: ow_lander/urdf/lander_lights.xacro (robot description, xacro)
@@ -1,5 +1,5 @@
 <?xml version="1.0"?>
 <robot xmlns:xacro="http://ros.org/wiki/xacro" name="lander_lights">
-  <xacro:macro name="lander_lights" params="lander_lights_parent_link off_x off_y off_z off_R off_P off_Y" >
+  <xacro:macro name="lander_lights" params="lander_lights_parent_link off_x off_y off_z off_R off_P off_Y vis_mask" >
     <link name="lander_lights_link" />
     <joint name="lander_lights_joint" type="fixed">
@@ -47,4 +47,9 @@
     <gazebo reference="lander_light${suffix}">
       <material>Gazebo/Grey</material>
+      <visual>
+        <plugin name="visibility" filename="libIRGVisibilityPlugin.so">
+          <visibility_bitmask>${vis_mask}</visibility_bitmask>
+        </plugin>
+      </visual>
       <light name="lander_light_light${suffix}" type="spot">
         <!-- Light is not transformed by the joint above, so we transform it here. -->

File: ow_lander/urdf/stereo_camera_triggered.xacro (robot description, xacro)
@@ -6,5 +6,5 @@
   <xacro:property name="camera_head_mass"   value="0.1" />
   <xacro:property name="deg_to_rad"         value="0.0174533" />
-  <xacro:macro name="stereo_camera" params="stereo_camera_parent_link hfov img_w img_h update_rate off_x off_y off_z off_R off_P off_Y">
+  <xacro:macro name="stereo_camera" params="stereo_camera_parent_link hfov img_w img_h update_rate off_x off_y off_z off_R off_P off_Y vis_mask">
   <link name="${Camera01Name}_head_link">
     <collision>
@@ -14,11 +14,11 @@
       </geometry>
     </collision>
-      <visual>
-        <origin xyz="0 0 0"  rpy="0 0 0"/>
-        <geometry>
-          <box size="0.025 ${camera_baseline} 0.025"/>
-        </geometry>
-        <material name="Gold"/>
-      </visual>
+    <visual>
+      <origin xyz="0 0 0"  rpy="0 0 0"/>
+      <geometry>
+        <box size="0.025 ${camera_baseline} 0.025"/>
+      </geometry>
+      <material name="Gold"/>
+    </visual>
     <visual>
       <origin xyz="0 ${camera_baseline/2} 0"  rpy="0 0 0"/>
@@ -50,4 +50,11 @@
     <origin xyz="${off_x} ${off_y} ${off_z}" rpy="${off_R} ${off_P} ${off_Y}" />
   </joint>
+  <gazebo reference="${Camera01Name}_head_link">
+    <visual>
+      <plugin name="visibility" filename="libIRGVisibilityPlugin.so">
+        <visibility_bitmask>${vis_mask}</visibility_bitmask>
+      </plugin>
+    </visual>
+  </gazebo>
   <!-- example for stereo setup is here: -->
   <!-- https://bitbucket.org/osrf/drcsim/src/52a691b8956045442ef22ba0aaee4520716807ff/multisense_sl_description/urdf/multisense_sl.urdf?at=default#cl-200 -->

Commit message: Squashed commit of the following:
commit 45c70536903c4ae15d095d64af54ac5431b9184b
Author: Mark B. Allan <Mark.B.Allan@nasa.gov>
Date:   Wed Oct 16 18:26:56 2019 -0700

    halt cmake if md5 sum fails

commit cb31631a23271b74d66c2cd60e5c2a005cdcd662
Merge: 0c16833 3367ca5
Author: Mark B. Allan <Mark.B.Allan@nasa.gov>
Date:   Wed Oct 16 10:48:42 2019 -0700

    Merge branch 'master' into feature/OCEANWATER-164

commit 0c168338d5daa74648c86d5456b555ef9b165fd0
Author: Mark B. Allan <Mark.B.Allan@nasa.gov>
Date:   Thu Oct 3 17:30:08 2019 -0700

    disable collision of scoop with terrain and add a link at tip of scoop that can be tracked for altitude above terrain

File: ow_lander/urdf/lander.xacro (robot description, xacro)
@@ -458,5 +458,5 @@
     <selfCollide>1</selfCollide>
     <!-- Turn off collisions with the terrain so scoop can go underground. For
-         this to work, the terrain must use a different collide_bitmask.
+         this to work, the terrain must use a different collide_bitmask.-->
     <collision>
       <surface>
@@ -466,5 +466,4 @@
       </surface>
     </collision>
-    -->
   </gazebo>
   <joint
@@ -547,5 +546,5 @@
     <selfCollide>1</selfCollide>
     <!-- Turn off collisions with the terrain so scoop can go underground. For
-         this to work, the terrain must use a different collide_bitmask.
+         this to work, the terrain must use a different collide_bitmask. -->
     <collision>
       <surface>
@@ -555,5 +554,21 @@
       </surface>
     </collision>
-    -->
+  </gazebo>
+  <!-- link that we can reference in Gazebo to get altitude of tip
+       of scoop above the terrain. Note that without an inertial
+       tag, the link will not show up in the SDF/Gazebo at all -->
+  <link name="l_scoop_tip">
+    <inertial>
+      <mass value="0.001"/>
+      <inertia ixx="1" ixy="0" ixz="0" iyy="1" iyz="0" izz="1"/>
+    </inertial>
+  </link>
+  <joint name="l_scoop_tip_joint" type="fixed">
+    <origin xyz="0.1 0.0 0.08" rpy="0 0 0"/>
+    <parent link="l_scoop"/>
+    <child link="l_scoop_tip"/>
+  </joint>
+  <gazebo reference="l_scoop_tip_joint">
+    <preserveFixedJoint>true</preserveFixedJoint>
   </gazebo>
   <joint

Commit message: Streamlined <script> tags with a xacro macro. Added path to light beam texture to fix lander lights.

File: ow_lander/urdf/lander.xacro (robot description, xacro)
@@ -21,4 +21,11 @@
     </joint>
   </xacro:if>
+  <xacro:macro name="material_script">
+    <script>
+      <uri>$(find ow_lander)/materials/scripts</uri>
+      <uri>$(find ow_europa)/models/terminator/materials/textures</uri>
+      <name>ow/lander</name>
+    </script>
+  </xacro:macro>
   <link name="base_link">
     <inertial>
@@ -65,8 +72,5 @@
         <diffuse>0.792 0.819 0.933 1</diffuse>
         <specular>0.4 0.4 0.4 1</specular>
-        <script>
-          <uri>package://ow_lander/materials/scripts</uri>
-          <name>ow/lander</name>
-        </script>
+        <xacro:material_script />
       </material>
       <plugin name="visibility" filename="libIRGVisibilityPlugin.so">
@@ -132,8 +136,5 @@
         <diffuse>0.898 0.917 0.929 1</diffuse>
         <specular>0.4 0.4 0.4 1</specular>
-        <script>
-          <uri>package://ow_lander/materials/scripts</uri>
-          <name>ow/lander</name>
-        </script>
+        <xacro:material_script />
       </material>
       <plugin name="visibility" filename="libIRGVisibilityPlugin.so">
@@ -211,8 +212,5 @@
         <diffuse>0.898 0.917 0.929 1</diffuse>
         <specular>0.4 0.4 0.4 1</specular>
-        <script>
-          <uri>package://ow_lander/materials/scripts</uri>
-          <name>ow/lander</name>
-        </script>
+        <xacro:material_script />
       </material>
       <plugin name="visibility" filename="libIRGVisibilityPlugin.so">
@@ -290,8 +288,5 @@
         <diffuse>0.898 0.917 0.929 1</diffuse>
         <specular>0.4 0.4 0.4 1</specular>
-        <script>
-          <uri>package://ow_lander/materials/scripts</uri>
-          <name>ow/lander</name>
-        </script>
+        <xacro:material_script />
       </material>
       <plugin name="visibility" filename="libIRGVisibilityPlugin.so">
@@ -369,8 +364,5 @@
         <diffuse>0.898 0.917 0.929 1</diffuse>
         <specular>0.4 0.4 0.4 1</specular>
-        <script>
-          <uri>package://ow_lander/materials/scripts</uri>
-          <name>ow/lander</name>
-        </script>
+        <xacro:material_script />
       </material>
       <plugin name="visibility" filename="libIRGVisibilityPlugin.so">
@@ -448,8 +440,5 @@
         <diffuse>0.898 0.917 0.929 1</diffuse>
         <specular>0.4 0.4 0.4 1</specular>
-        <script>
-          <uri>package://ow_lander/materials/scripts</uri>
-          <name>ow/lander</name>
-        </script>
+        <xacro:material_script />
       </material>
       <plugin name="visibility" filename="libIRGVisibilityPlugin.so">
@@ -536,8 +525,5 @@
         <diffuse>0.898 0.917 0.929 1</diffuse>
         <specular>0.4 0.4 0.4 1</specular>
-        <script>
-          <uri>package://ow_lander/materials/scripts</uri>
-          <name>ow/lander</name>
-        </script>
+        <xacro:material_script />
       </material>
       <plugin name="visibility" filename="libIRGVisibilityPlugin.so">
@@ -641,8 +627,5 @@
         <diffuse>0.294 0.294 0.294 1</diffuse>
         <specular>0.4 0.4 0.4 1</specular>
-        <script>
-          <uri>package://ow_lander/materials/scripts</uri>
-          <name>ow/lander</name>
-        </script>
+        <xacro:material_script />
       </material>
       <plugin name="visibility" filename="libIRGVisibilityPlugin.so">
@@ -720,8 +703,5 @@
         <diffuse>0.294 0.294 0.294 1</diffuse>
         <specular>0.4 0.4 0.4 1</specular>
-        <script>
-          <uri>package://ow_lander/materials/scripts</uri>
-          <name>ow/lander</name>
-        </script>
+        <xacro:material_script />
       </material>
       <plugin name="visibility" filename="libIRGVisibilityPlugin.so">
