Commit message: New moments of intertia and some new masses for the arm.

File: ow_lander/urdf/lander.xacro (robot description, xacro)
@@ -98,12 +98,12 @@
         rpy="0 0 0" />
       <mass
-        value="7.02920774782214" />
-      <inertia
-        ixx="0.0104575300282247"
-        ixy="-0.000601021251095754"
-        ixz="-0.00827528301657843"
-        iyy="0.0383526039269065"
-        iyz="-0.000231653878395009"
-        izz="0.0311579762615783" />
+        value="7.0292" />
+      <inertia
+        ixx="0.024707226"
+        ixy="0.001106126"
+        ixz="0.008780403"
+        iyy="0.053430638"
+        iyz="0.000231645"
+        izz="0.050909058" />
     </inertial>
     <visual>
@@ -174,12 +174,12 @@
         rpy="0 0 0" />
       <mass
-        value="4.19335228756063" />
-      <inertia
-        ixx="0.010970201330525"
-        ixy="-1.57434663712407E-07"
-        ixz="0.00200163732633334"
-        iyy="0.134978241858844"
-        iyz="1.14891258563061E-18"
-        izz="0.124008040530309" />
+        value="3.98552" />
+      <inertia
+        ixx="0.010948108"
+        ixy="0.000000123"
+        ixz="-0.016431513"
+        iyy="0.140543709"
+        iyz="0"
+        izz="0.141291863" />
     </inertial>
     <visual>
@@ -250,12 +250,12 @@
         rpy="0 0 0" />
       <mass
-        value="3.47049693100743" />
-      <inertia
-        ixx="0.00621200133375043"
-        ixy="-7.94830322787864E-08"
-        ixz="-0.0264356399717985"
-        iyy="0.444337175366728"
-        iyz="2.25893478477412E-17"
-        izz="0.43812517403302" />
+        value="3.4705" />
+      <inertia
+        ixx="0.02219061"
+        ixy="0.000000071"
+        ixz="0.0217064.66"
+        iyy="0.50510019"
+        iyz="0"
+        izz="0.497745918" />
     </inertial>
     <visual>
@@ -326,12 +326,12 @@
         rpy="0 0 0" />
       <mass
-        value="1.24254588886639" />
-      <inertia
-        ixx="0.00600454075116932"
-        ixy="-0.000821319339321742"
-        ixz="-0.00975159245248633"
-        iyy="0.0288075930851101"
-        iyz="-0.000314668908607835"
-        izz="0.0262750836489082" />
+        value="1.2425" />
+      <inertia
+        ixx="0.013575388"
+        ixy="-0.000000011"
+        ixz="0.010276112"
+        iyy="0.041535122"
+        iyz="0.00000001"
+        izz="0.040985679" />
     </inertial>
     <visual>
@@ -402,12 +402,12 @@
         rpy="0 0 0" />
       <mass
-        value="1.08554586923443" />
-      <inertia
-        ixx="0.00868815536634117"
-        ixy="-7.25951344207531E-09"
-        ixz="-0.000954522050362788"
-        iyy="0.00879302369591146"
-        iyz="-6.60768189073236E-08"
-        izz="0.000104868330575369" />
+        value="1.0855" />
+      <inertia
+        ixx="0.031145341"
+        ixy="-0.000000019"
+        ixz="0.000003178"
+        iyy="0.03114165"
+        iyz="0.000000034"
+        izz="0.021681969" />
     </inertial>
     <visual>
@@ -487,12 +487,12 @@
         rpy="0 0 0" />
       <mass
-        value="0.191928708332057" />
-      <inertia
-        ixx="0.0128625280820728"
-        ixy="-0.0550577074342039"
-        ixz="4.59706499938512E-09"
-        iyy="0.252496809842602"
-        iyz="4.83511231053058E-10"
-        izz="0.265359337924673" />
+        value="0.30936" />
+      <inertia
+        ixx="0.001031142"
+        ixy="0"
+        ixz="0.000157564"
+        iyy="0.001225161"
+        iyz="0"
+        izz="0.000591262" />
     </inertial>
     <visual>

Commit message: Camera and lights use the same shader material as lander. Removed a little legacy code and tweaked camera and light positions.

File: ow_lander/urdf/lander.xacro (robot description, xacro)
@@ -5,9 +5,9 @@
   <xacro:stereo_camera stereo_camera_parent_link="l_ant_panel"
                      hfov="21" img_w="1600" img_h="1200" update_rate="1"
-                     off_x="0.55" off_y="0.05" off_z="0.0" off_R="${pi/2.0}" off_P="${pi}" off_Y="${pi/2.0}"
+                     off_x="0.53811" off_y="0.07" off_z="0.0" off_R="${pi/2.0}" off_P="${pi}" off_Y="${pi/2.0}"
                      vis_mask="${vis_mask}" />
   <xacro:include filename="$(find ow_lander)/urdf/lander_lights.xacro" />
   <xacro:lander_lights lander_lights_parent_link="l_ant_panel"
-                     off_x="0.85" off_y="0.07" off_z="0.0" off_R="-${pi/2.0}" off_P="0.0" off_Y="0.0"
+                     off_x="0.85" off_y="0.08" off_z="0.0" off_R="-${pi/2.0}" off_P="0.0" off_Y="0.0"
                      vis_mask="${vis_mask}" />
   <xacro:arg name="freeze_base_link" default="false"/>
@@ -21,11 +21,4 @@
     </joint>
   </xacro:if>
-  <xacro:macro name="material_script">
-    <script>
-      <uri>$(find ow_lander)/materials/scripts</uri>
-      <uri>$(find ow_europa)/models/terminator/materials/textures</uri>
-      <name>ow/lander</name>
-    </script>
-  </xacro:macro>
   <link name="base_link">
     <inertial>

File: ow_lander/urdf/lander_lights.xacro (robot description, xacro)
@@ -1,4 +1,5 @@
 <?xml version="1.0"?>
 <robot xmlns:xacro="http://ros.org/wiki/xacro" name="lander_lights">
+  <xacro:include filename="$(find ow_lander)/urdf/material_script.xacro" />
   <xacro:macro name="lander_lights" params="lander_lights_parent_link off_x off_y off_z off_R off_P off_Y vis_mask" >
     <link name="lander_lights_link" />
@@ -30,4 +31,7 @@
           <cylinder length="0.05" radius="0.03" />
         </geometry>
+        <material name="">
+          <color rgba="0.7 0.7 0.7 1" />
+        </material>
       </visual>
       <inertial>
@@ -46,6 +50,10 @@
     </joint>
     <gazebo reference="lander_light${suffix}">
-      <material>Gazebo/Grey</material>
       <visual>
+        <material>
+          <diffuse>0.7 0.7 0.7 1</diffuse>
+          <specular>0.4 0.4 0.4 1</specular>
+          <xacro:material_script />
+        </material>
         <plugin name="visibility" filename="libIRGVisibilityPlugin.so">
           <visibility_bitmask>${vis_mask}</visibility_bitmask>

File: ow_lander/urdf/stereo_camera_triggered.xacro (robot description, xacro)
@@ -6,4 +6,5 @@
   <xacro:property name="camera_head_mass"   value="0.1" />
   <xacro:property name="deg_to_rad"         value="0.0174533" />
+  <xacro:include filename="$(find ow_lander)/urdf/material_script.xacro" />
   <xacro:macro name="stereo_camera" params="stereo_camera_parent_link hfov img_w img_h update_rate off_x off_y off_z off_R off_P off_Y vis_mask">
   <link name="${Camera01Name}_head_link">
@@ -19,5 +20,7 @@
         <box size="0.025 ${camera_baseline} 0.025"/>
       </geometry>
-      <material name="Gold"/>
+      <material name="">
+        <color rgba="0.9 0.7 0.2 1" />
+      </material>
     </visual>
     <visual>
@@ -26,5 +29,7 @@
         <box size="0.1 0.1 0.1"/>
       </geometry>
-      <material name="Gold"/>
+      <material name="">
+        <color rgba="0.9 0.7 0.2 1" />
+      </material>
     </visual>
     <visual>
@@ -33,10 +38,11 @@
         <box size="0.1 0.1 0.1"/>
       </geometry>
-      <material name="Gold"/>
+      <material name="">
+        <color rgba="0.9 0.7 0.2 1" />
+      </material>
     </visual>
     <inertial>
       <mass value="${camera_head_mass}" />
       <origin xyz="0 0 0" rpy="0 0 0"/>
-      <!-- inertia ixx="0.05" ixy="0" ixz="0" iyy="0.05" iyz="0" izz="0.05" / -->
       <inertia
           ixx="${camera_head_mass / 12.0 * (camera_baseline*camera_baseline + 0.1*0.1)}" ixy="0.0" ixz="0.0"
@@ -52,4 +58,9 @@
   <gazebo reference="${Camera01Name}_head_link">
     <visual>
+      <material>
+        <diffuse>0.9 0.7 0.2 1</diffuse>
+        <specular>0.4 0.4 0.4 1</specular>
+        <xacro:material_script />
+      </material>
       <plugin name="visibility" filename="libIRGVisibilityPlugin.so">
         <visibility_bitmask>${vis_mask}</visibility_bitmask>
@@ -60,5 +71,4 @@
   <!-- https://bitbucket.org/osrf/drcsim/src/52a691b8956045442ef22ba0aaee4520716807ff/multisense_sl_description/urdf/multisense_sl.urdf?at=default#cl-200 -->
   <!-- https://bitbucket.org/osrf/drcsim/src/52a691b8956045442ef22ba0aaee4520716807ff/drcsim_gazebo/launch/atlas_bringup.launch?at=default#cl-38 -->
-  <gazebo reference="${Camera01Name}Left_link"/>
   <link name="${Camera01Name}Left_link"/>
   <link name="${Camera01Name}Left_optical_frame"/>
@@ -73,5 +83,4 @@
     <child link="${Camera01Name}Left_optical_frame"/>
   </joint>
-  <gazebo reference="${Camera01Name}Right_link"/>
   <link name="${Camera01Name}Right_link"/>
   <link name="${Camera01Name}Right_optical_frame"/>
@@ -87,5 +96,4 @@
   </joint>
   <gazebo reference="${Camera01Name}Left_link">
-    <material>Gazebo/Red</material>
     <sensor type="multicamera" name="${Camera01Name}">
       <update_rate>${update_rate}</update_rate>
@@ -139,5 +147,4 @@
   </gazebo>
   <!-- "Center Camera" for "video" -->
-  <gazebo reference="${Camera01Name}Center_link"/>
   <link name="${Camera01Name}Center_link"/>
   <link name="${Camera01Name}Center_optical_frame"/>
@@ -159,6 +166,4 @@
         <horizontal_fov>${hfov*deg_to_rad}</horizontal_fov>
         <image>
-          <!--width>1280</width>
-          <height>720</height -->
           <width>${img_w/2}</width>
           <height>${img_h/2}</height>

Commit message: Lander uses LinkForcePlugin.

File: ow_lander/urdf/lander.xacro (robot description, xacro)
@@ -738,4 +738,8 @@
       <updateRate>10</updateRate>
     </plugin-->
+    <plugin name="LinkForce" filename="libLinkForcePlugin.so">
+      <link>l_scoop</link>
+      <lookupTable>$(find ow_gazebo_plugins)/data/scoop_force_circular.csv</lookupTable>
+    </plugin>
   </gazebo>
 </robot>

Commit message: CosimulatorPlugin added to lander.xacro and error handling cleaned up.

File: ow_lander/urdf/lander.xacro (robot description, xacro)
@@ -738,4 +738,25 @@
       <updateRate>10</updateRate>
     </plugin-->
+    <plugin name="CosimulationPlugin" filename="libCosimulationPlugin.so">
+      <!-- all parameters given in SI units -->
+      <!-- link_ and particle_ are set to the same values used in EDEM sim -->
+      <link>l_scoop</link>
+      <link_model>l_scoop.STL</link_model>
+      <link_youngs_modulus>6.9e10</link_youngs_modulus>
+      <link_poisson_ratio>0.33</link_poisson_ratio>
+      <link_restitution_coef>0.7</link_restitution_coef>
+      <link_static_friction_coef>0.58</link_static_friction_coef>
+      <link_rolling_friction_coef>0.05</link_rolling_friction_coef>
+      <particle_youngs_modulus>2.72e7</particle_youngs_modulus>
+      <particle_poisson_ratio>0.36</particle_poisson_ratio>
+      <particle_restitution_coef>0.88</particle_restitution_coef>
+      <particle_static_friction_coef>0.58</particle_static_friction_coef>
+      <particle_rolling_friction_coef>0.05</particle_rolling_friction_coef>
+      <particle_density>300</particle_density>
+      <particle_radius>1.75e-3</particle_radius>
+      <workspace_dimensions>0.5 0.5 0.2</workspace_dimensions>
+      <workspace_pose>0 0 0 1 0 0 0</workspace_pose>
+      <timestep>1e-6</timestep>
+    </plugin>
   </gazebo>
 </robot>

Commit message: Added README.md to CosimulationPlugin and class summarizing comments.
Also removed the CosimulationPlugin's implementation from the
lander.xacro file since it may collide with another plugin already
merged with master, and its implmentation is now captured in the
README.md.

File: ow_lander/urdf/lander.xacro (robot description, xacro)
@@ -738,25 +738,4 @@
       <updateRate>10</updateRate>
     </plugin-->
-    <plugin name="CosimulationPlugin" filename="libCosimulationPlugin.so">
-      <!-- all parameters given in SI units -->
-      <!-- link_ and particle_ are set to the same values used in EDEM sim -->
-      <link>l_scoop</link>
-      <link_model>l_scoop.STL</link_model>
-      <link_youngs_modulus>6.9e10</link_youngs_modulus>
-      <link_poisson_ratio>0.33</link_poisson_ratio>
-      <link_restitution_coef>0.7</link_restitution_coef>
-      <link_static_friction_coef>0.58</link_static_friction_coef>
-      <link_rolling_friction_coef>0.05</link_rolling_friction_coef>
-      <particle_youngs_modulus>2.72e7</particle_youngs_modulus>
-      <particle_poisson_ratio>0.36</particle_poisson_ratio>
-      <particle_restitution_coef>0.88</particle_restitution_coef>
-      <particle_static_friction_coef>0.58</particle_static_friction_coef>
-      <particle_rolling_friction_coef>0.05</particle_rolling_friction_coef>
-      <particle_density>300</particle_density>
-      <particle_radius>1.75e-3</particle_radius>
-      <workspace_dimensions>0.5 0.5 0.2</workspace_dimensions>
-      <workspace_pose>0 0 0 1 0 0 0</workspace_pose>
-      <timestep>1e-6</timestep>
-    </plugin>
   </gazebo>
 </robot>

Commit message: Added simple grinder end effector.

File: ow_lander/urdf/lander.xacro (robot description, xacro)
@@ -576,4 +576,73 @@
     </actuator>
   </transmission>
+  <link name="l_grinder">
+    <inertial>
+      <origin
+        xyz="0 0 0.06"
+        rpy="0 0 0" />
+      <mass
+        value="0.5" />
+      <inertia
+        ixx="0.002"
+        ixy="0"
+        ixz="0"
+        iyy="0.002"
+        iyz="0"
+        izz="0.002" />
+    </inertial>
+    <visual>
+      <origin
+        xyz="0 0 0"
+        rpy="0 0 0" />
+      <geometry>
+        <mesh
+          filename="package://ow_lander/meshes/l_grinder.STL" />
+      </geometry>
+      <material
+        name="">
+        <color
+          rgba="0.6 0.6 0.6 1" />
+      </material>
+    </visual>
+    <collision>
+      <origin
+        xyz="0 0 0"
+        rpy="0 0 0" />
+      <geometry>
+        <mesh
+          filename="package://ow_lander/meshes/l_grinder.STL" />
+      </geometry>
+    </collision>
+  </link>
+  <gazebo reference="l_grinder">
+    <visual>
+      <material>
+        <diffuse>0.6 0.6 0.6 1</diffuse>
+        <specular>0.2 0.2 0.2 1</specular>
+        <xacro:material_script />
+      </material>
+      <plugin name="visibility" filename="libIRGVisibilityPlugin.so">
+        <visibility_bitmask>${vis_mask}</visibility_bitmask>
+      </plugin>
+    </visual>
+    <selfCollide>1</selfCollide>
+    <!-- Turn off collisions with the terrain so scoop can go underground. For
+         this to work, the terrain must use a different collide_bitmask. -->
+    <collision>
+      <surface>
+        <contact>
+          <collide_bitmask>0x0002</collide_bitmask>
+        </contact>
+      </surface>
+    </collision>
+  </gazebo>
+  <joint name="j_grinder" type="fixed">
+    <origin xyz="-0.075 -0.129903811 0" rpy="0 0 ${-pi*2/3}" />
+    <parent link="l_hand" />
+    <child link="l_grinder" />
+  </joint>
+  <gazebo reference="j_grinder">
+    <preserveFixedJoint>true</preserveFixedJoint>
+  </gazebo>
   <link name="l_ant_foot">
     <inertial>

Commit message: Tuned PID-controller gains, reduced joints' maximum velocities to prevent hand from hanging up on leg

File: ow_lander/urdf/lander.xacro (robot description, xacro)
@@ -153,6 +153,6 @@
     <axis
       xyz="0 0 -1" />
-    <dynamics damping="50" />
-    <limit effort="1000.0" velocity="0.4" lower="-1.8" upper="1.8"/>
+    <dynamics damping="50.0" />
+    <limit effort="1000.0" velocity="0.15" lower="-1.8" upper="1.8"/>
   </joint>
   <transmission name="shou_yaw_transmission">
@@ -229,6 +229,6 @@
     <axis
       xyz="0 0 -1" />
-    <dynamics damping="50" />
-    <limit effort="1000.0" velocity="0.4" lower="0.05" upper="2.2"/>
+    <dynamics damping="50.0" />
+    <limit effort="1000.0" velocity="0.2" lower="0.05" upper="2.2"/>
   </joint>
   <transmission name="shou_pitch_transmission">
@@ -305,6 +305,6 @@
     <axis
       xyz="0 0 -1" />
-    <dynamics damping="50" />
-    <limit effort="1000.0" velocity="0.4" />
+    <dynamics damping="50.0" />
+    <limit effort="1000.0" velocity="0.2" />
   </joint>
   <transmission name="prox_pitch_transmission">
@@ -381,6 +381,6 @@
     <axis
       xyz="0 0 1" />
-    <dynamics damping="50" />
-    <limit effort="1000.0" velocity="0.4" />
+    <dynamics damping="50.0" />
+    <limit effort="1000.0" velocity="0.2" />
   </joint>
   <transmission name="dist_pitch_transmission">
@@ -466,6 +466,6 @@
     <axis
       xyz="0 0 -1" />
-    <dynamics damping="50" />
-    <limit effort="1000.0" velocity="0.4" />
+    <dynamics damping="50.0" />
+    <limit effort="1000.0" velocity="0.2" />
   </joint>
   <transmission name="hand_yaw_transmission">

Commit message: New service start_unstowed plus new PID and velocities values

File: ow_lander/urdf/lander.xacro (robot description, xacro)
@@ -154,5 +154,5 @@
       xyz="0 0 -1" />
     <dynamics damping="50" />
-    <limit effort="1000.0" velocity="0.4" lower="-1.8" upper="1.8"/>
+    <limit effort="1000.0" velocity="0.2" lower="-1.8" upper="1.8"/>
   </joint>
   <transmission name="shou_yaw_transmission">
@@ -230,5 +230,5 @@
       xyz="0 0 -1" />
     <dynamics damping="50" />
-    <limit effort="1000.0" velocity="0.4" lower="0.05" upper="2.2"/>
+    <limit effort="1000.0" velocity="0.2" lower="0.05" upper="2.2"/>
   </joint>
   <transmission name="shou_pitch_transmission">
@@ -306,5 +306,5 @@
       xyz="0 0 -1" />
     <dynamics damping="50" />
-    <limit effort="1000.0" velocity="0.4" />
+    <limit effort="1000.0" velocity="0.2" />
   </joint>
   <transmission name="prox_pitch_transmission">
@@ -382,5 +382,5 @@
       xyz="0 0 1" />
     <dynamics damping="50" />
-    <limit effort="1000.0" velocity="0.4" />
+    <limit effort="1000.0" velocity="0.2" />
   </joint>
   <transmission name="dist_pitch_transmission">
@@ -467,5 +467,5 @@
       xyz="0 0 -1" />
     <dynamics damping="50" />
-    <limit effort="1000.0" velocity="0.4" />
+    <limit effort="1000.0" velocity="0.2" />
   </joint>
   <transmission name="hand_yaw_transmission">
@@ -569,5 +569,5 @@
       xyz="0 0 -1" />
     <dynamics damping="50" />
-    <limit effort="1000.0" velocity="0.4" />
+    <limit effort="1000.0" velocity="0.2" />
   </joint>
   <transmission name="scoop_yaw_transmission">
@@ -714,5 +714,5 @@
       xyz="0 0 -1" />
     <dynamics damping="50" />
-    <limit effort="1000.0" velocity="0.4" />
+    <limit effort="1000.0" velocity="0.2" />
   </joint>
   <transmission name="ant_pan_transmission">
@@ -790,5 +790,5 @@
       xyz="0 0 -1" />
     <dynamics damping="50" />
-    <limit effort="1000.0" velocity="0.4" />
+    <limit effort="1000.0" velocity="0.2" />
   </joint>
   <transmission name="ant_tilt_transmission">

Commit message: Changed PID values to avoid vibration

File: ow_lander/urdf/lander.xacro (robot description, xacro)
@@ -531,5 +531,5 @@
     <!-- Turn off collisions with the terrain so scoop can go underground. For
          this to work, the terrain must use a different collide_bitmask. -->
-    <collision>
+    <!--collision>
       <surface>
         <contact>
@@ -537,5 +537,5 @@
         </contact>
       </surface>
-    </collision>
+    </collision-->
   </gazebo>
   <!-- link that we can reference in Gazebo to get altitude of tip

Commit message: Reduced gains to avoid vibrations

File: ow_lander/urdf/lander.xacro (robot description, xacro)
@@ -531,5 +531,5 @@
     <!-- Turn off collisions with the terrain so scoop can go underground. For
          this to work, the terrain must use a different collide_bitmask. -->
-    <!--collision>
+    <collision>
       <surface>
         <contact>
@@ -537,5 +537,5 @@
         </contact>
       </surface>
-    </collision-->
+    </collision>
   </gazebo>
   <!-- link that we can reference in Gazebo to get altitude of tip

Commit message: Unstowed service

File: ow_lander/urdf/lander.xacro (robot description, xacro)
@@ -154,5 +154,5 @@
       xyz="0 0 -1" />
     <dynamics damping="50" />
-    <limit effort="1000.0" velocity="0.2" lower="-1.8" upper="1.8"/>
+    <limit effort="1000.0" velocity="0.4" lower="-1.8" upper="1.8"/>
   </joint>
   <transmission name="shou_yaw_transmission">
@@ -230,5 +230,5 @@
       xyz="0 0 -1" />
     <dynamics damping="50" />
-    <limit effort="1000.0" velocity="0.2" lower="0.05" upper="2.2"/>
+    <limit effort="1000.0" velocity="0.4" lower="0.05" upper="2.2"/>
   </joint>
   <transmission name="shou_pitch_transmission">
@@ -306,5 +306,5 @@
       xyz="0 0 -1" />
     <dynamics damping="50" />
-    <limit effort="1000.0" velocity="0.2" />
+    <limit effort="1000.0" velocity="0.4" />
   </joint>
   <transmission name="prox_pitch_transmission">
@@ -382,5 +382,5 @@
       xyz="0 0 1" />
     <dynamics damping="50" />
-    <limit effort="1000.0" velocity="0.2" />
+    <limit effort="1000.0" velocity="0.4" />
   </joint>
   <transmission name="dist_pitch_transmission">
@@ -467,5 +467,5 @@
       xyz="0 0 -1" />
     <dynamics damping="50" />
-    <limit effort="1000.0" velocity="0.2" />
+    <limit effort="1000.0" velocity="0.4" />
   </joint>
   <transmission name="hand_yaw_transmission">
@@ -569,5 +569,5 @@
       xyz="0 0 -1" />
     <dynamics damping="50" />
-    <limit effort="1000.0" velocity="0.2" />
+    <limit effort="1000.0" velocity="0.4" />
   </joint>
   <transmission name="scoop_yaw_transmission">
@@ -714,5 +714,5 @@
       xyz="0 0 -1" />
     <dynamics damping="50" />
-    <limit effort="1000.0" velocity="0.2" />
+    <limit effort="1000.0" velocity="0.4" />
   </joint>
   <transmission name="ant_pan_transmission">
@@ -790,5 +790,5 @@
       xyz="0 0 -1" />
     <dynamics damping="50" />
-    <limit effort="1000.0" velocity="0.2" />
+    <limit effort="1000.0" velocity="0.4" />
   </joint>
   <transmission name="ant_tilt_transmission">

Commit message: use velocity instead of effort

File: ow_lander/urdf/lander.xacro (robot description, xacro)
@@ -535,5 +535,5 @@
     <!-- Turn off collisions with the terrain so scoop can go underground. For
          this to work, the terrain must use a different collide_bitmask. -->
-    <collision>
+    <!--collision>
       <surface>
         <contact>
@@ -541,5 +541,5 @@
         </contact>
       </surface>
-    </collision>
+    </collision-->
   </gazebo>
   <!-- link that we can reference in Gazebo to get altitude of tip

Commit message: answers to comments

File: ow_lander/urdf/lander.xacro (robot description, xacro)
@@ -535,5 +535,5 @@
     <!-- Turn off collisions with the terrain so scoop can go underground. For
          this to work, the terrain must use a different collide_bitmask. -->
-    <!--collision>
+    <collision>
       <surface>
         <contact>
@@ -541,5 +541,5 @@
         </contact>
       </surface>
-    </collision-->
+    </collision>
   </gazebo>
   <!-- link that we can reference in Gazebo to get altitude of tip
