Commit message: Working implmenentation for different topics

File: ow_lander/urdf/lander.xacro (robot description, xacro)
@@ -533,13 +533,4 @@
     </visual>
     <selfCollide>1</selfCollide>
-    <!-- Turn off collisions with the terrain so scoop can go underground. For
-         this to work, the terrain must use a different collide_bitmask. -->
-    <collision>
-      <surface>
-        <contact>
-          <collide_bitmask>0x0002</collide_bitmask>
-        </contact>
-      </surface>
-    </collision>
   </gazebo>
   <!-- link that we can reference in Gazebo to get altitude of tip
@@ -635,13 +626,4 @@
     </visual>
     <selfCollide>1</selfCollide>
-    <!-- Turn off collisions with the terrain so scoop can go underground. For
-         this to work, the terrain must use a different collide_bitmask. -->
-    <collision>
-      <surface>
-        <contact>
-          <collide_bitmask>0x0002</collide_bitmask>
-        </contact>
-      </surface>
-    </collision>
   </gazebo>
   <joint name="j_grinder" type="fixed">

Commit message: Disable grinder collision + document some aspects of the code + code formatting + add the notices and disclaimers header

File: ow_lander/urdf/lander.xacro (robot description, xacro)
@@ -626,4 +626,11 @@
     </visual>
     <selfCollide>1</selfCollide>
+    <collision>
+      <surface>
+        <contact>
+          <collide_bitmask>0x0002</collide_bitmask>
+        </contact>
+      </surface>
+    </collision>
   </gazebo>
   <joint name="j_grinder" type="fixed">

Commit message: Tuned PID, tried to eliminate jerking motion

File: ow_lander/urdf/lander.xacro (robot description, xacro)
@@ -158,5 +158,5 @@
       xyz="0 0 -1" />
     <dynamics damping="50.0" />
-    <limit effort="1000.0" velocity="0.15" lower="-1.8" upper="1.8"/>
+    <limit effort="100.0" velocity="0.15" lower="-1.8" upper="1.8"/>
   </joint>
   <transmission name="shou_yaw_transmission">
@@ -234,5 +234,5 @@
       xyz="0 0 -1" />
     <dynamics damping="50.0" />
-    <limit effort="1000.0" velocity="0.2" lower="0.05" upper="2.2"/>
+    <limit effort="100.0" velocity="0.2" lower="0.05" upper="2.2"/>
   </joint>
   <transmission name="shou_pitch_transmission">
@@ -310,5 +310,5 @@
       xyz="0 0 -1" />
     <dynamics damping="50.0" />
-    <limit effort="1000.0" velocity="0.2" />
+    <limit effort="100.0" velocity="0.2" />
   </joint>
   <transmission name="prox_pitch_transmission">
@@ -386,5 +386,5 @@
       xyz="0 0 1" />
     <dynamics damping="50.0" />
-    <limit effort="1000.0" velocity="0.2" />
+    <limit effort="100.0" velocity="0.2" />
   </joint>
   <transmission name="dist_pitch_transmission">
@@ -471,5 +471,5 @@
       xyz="0 0 -1" />
     <dynamics damping="50.0" />
-    <limit effort="1000.0" velocity="0.2" />
+    <limit effort="50.0" velocity="0.2" />
   </joint>
   <transmission name="hand_yaw_transmission">
@@ -573,5 +573,5 @@
       xyz="0 0 -1" />
     <dynamics damping="50" />
-    <limit effort="1000.0" velocity="0.4" />
+    <limit effort="30.0" velocity="0.4" />
   </joint>
   <transmission name="scoop_yaw_transmission">

Commit message: Ensure same digging values works for all terrains + Grinder only affects 1/3 of the value + Enable collision for scoop and grinder

File: ow_lander/urdf/lander.xacro (robot description, xacro)
@@ -533,4 +533,11 @@
     </visual>
     <selfCollide>1</selfCollide>
+    <collision>
+      <surface>
+        <contact>
+          <collide_bitmask>0x0001</collide_bitmask>
+        </contact>
+      </surface>
+    </collision>
   </gazebo>
   <!-- link that we can reference in Gazebo to get altitude of tip
@@ -629,5 +636,5 @@
       <surface>
         <contact>
-          <collide_bitmask>0x0002</collide_bitmask>
+          <collide_bitmask>0x0001</collide_bitmask>
         </contact>
       </surface>

Commit message: Grinder keeps vertical, added revolute joint and controller to grinder, created grinder motion group, changed radial with parallel, non-parallel griding works, changed defaults.

File: ow_lander/urdf/lander.xacro (robot description, xacro)
@@ -641,12 +641,23 @@
     </collision>
   </gazebo>
-  <joint name="j_grinder" type="fixed">
+  <joint
+    name="j_grinder"
+    type="revolute">
     <origin xyz="-0.075 -0.129903811 0" rpy="0 0 ${-pi*2/3}" />
     <parent link="l_hand" />
     <child link="l_grinder" />
-  </joint>
-  <gazebo reference="j_grinder">
-    <preserveFixedJoint>true</preserveFixedJoint>
-  </gazebo>
+    <axis xyz="-1 0 0" />
+    <dynamics damping="1" />
+    <limit lower="-3.14" upper="3.14" effort="1.0" velocity="0.1" />
+  </joint>
+  <transmission name="grinder_yaw_transmission">
+    <type>transmission_interface/SimpleTransmission</type>
+    <joint name="j_grinder">
+      <hardwareInterface>hardware_interface/EffortJointInterface</hardwareInterface>
+    </joint>
+    <actuator name="grinder_yaw_motor">
+      <mechanicalReduction>1</mechanicalReduction>
+    </actuator>
+  </transmission>
   <link name="l_ant_foot">
     <inertial>

Commit message: removed link-force plugin

File: ow_lander/urdf/lander.xacro (robot description, xacro)
@@ -822,8 +822,4 @@
       <updateRate>10</updateRate>
     </plugin-->
-    <plugin name="LinkForce" filename="libLinkForcePlugin.so">
-      <link>l_scoop</link>
-      <lookupTable>$(find ow_gazebo_plugins)/data/scoop_force_circular.csv</lookupTable>
-    </plugin>
   </gazebo>
 </robot>

Commit message: 1)Added parameters to stabilize scoop-terrain interaction, 2)Added realistic values of friction and maximum torque to joints

File: ow_lander/urdf/lander.xacro (robot description, xacro)
@@ -157,6 +157,6 @@
     <axis
       xyz="0 0 -1" />
-    <dynamics damping="50.0" />
-    <limit effort="100.0" velocity="0.15" lower="-1.8" upper="1.8"/>
+    <dynamics damping="50.0" friction="5.1"/>
+    <limit effort="50.9" velocity="0.2" lower="-1.8" upper="1.8"/>
   </joint>
   <transmission name="shou_yaw_transmission">
@@ -233,6 +233,6 @@
     <axis
       xyz="0 0 -1" />
-    <dynamics damping="50.0" />
-    <limit effort="100.0" velocity="0.2" lower="0.05" upper="2.2"/>
+    <dynamics damping="50.0" friction="9.1"/>
+    <limit effort="91.0" velocity="0.2" lower="0.05" upper="2.2"/>
   </joint>
   <transmission name="shou_pitch_transmission">
@@ -309,6 +309,6 @@
     <axis
       xyz="0 0 -1" />
-    <dynamics damping="50.0" />
-    <limit effort="100.0" velocity="0.2" />
+    <dynamics damping="50.0" friction="5.3"/>
+    <limit effort="53.0" velocity="0.2"/>
   </joint>
   <transmission name="prox_pitch_transmission">
@@ -385,6 +385,6 @@
     <axis
       xyz="0 0 1" />
-    <dynamics damping="50.0" />
-    <limit effort="100.0" velocity="0.2" />
+    <dynamics damping="50.0" friction="0.6"/>
+    <limit effort="5.7" velocity="0.2" />
   </joint>
   <transmission name="dist_pitch_transmission">
@@ -470,6 +470,6 @@
     <axis
       xyz="0 0 -1" />
-    <dynamics damping="50.0" />
-    <limit effort="50.0" velocity="0.2" />
+    <dynamics damping="50.0" friction="0.6"/>
+    <limit effort="5.7" velocity="0.2" />
   </joint>
   <transmission name="hand_yaw_transmission">
@@ -537,4 +537,8 @@
         <contact>
           <collide_bitmask>0x0001</collide_bitmask> <!-- Enable collision with the terrain by matching the bitmask -->
+          <ode>
+            <kp>1e+15</kp>
+            <kd>1e+13</kd>
+          </ode>
         </contact>
       </surface>
@@ -570,6 +574,6 @@
     <axis
       xyz="0 0 -1" />
-    <dynamics damping="50" />
-    <limit effort="30.0" velocity="0.4" />
+    <dynamics damping="50.0" friction="1.0"/>
+    <limit effort="10.0" velocity="0.2" />
   </joint>
   <transmission name="scoop_yaw_transmission">

Commit message: Reverted unwanted change on shou_yaw velocity limit

File: ow_lander/urdf/lander.xacro (robot description, xacro)
@@ -158,5 +158,5 @@
       xyz="0 0 -1" />
     <dynamics damping="50.0" friction="5.1"/>
-    <limit effort="50.9" velocity="0.2" lower="-1.8" upper="1.8"/>
+    <limit effort="50.9" velocity="0.15" lower="-1.8" upper="1.8"/>
   </joint>
   <transmission name="shou_yaw_transmission">

Commit message: Increased effort limit, decreased friction torque

File: ow_lander/urdf/lander.xacro (robot description, xacro)
@@ -157,6 +157,6 @@
     <axis
       xyz="0 0 -1" />
-    <dynamics damping="50.0" friction="5.1"/>
-    <limit effort="50.9" velocity="0.15" lower="-1.8" upper="1.8"/>
+    <dynamics damping="50.0" friction="2.6"/>
+    <limit effort="70.9" velocity="0.15" lower="-1.8" upper="1.8"/>
   </joint>
   <transmission name="shou_yaw_transmission">
@@ -233,6 +233,6 @@
     <axis
       xyz="0 0 -1" />
-    <dynamics damping="50.0" friction="9.1"/>
-    <limit effort="91.0" velocity="0.2" lower="0.05" upper="2.2"/>
+    <dynamics damping="50.0" friction="4.6"/>
+    <limit effort="101.0" velocity="0.2" lower="0.05" upper="2.2"/>
   </joint>
   <transmission name="shou_pitch_transmission">
@@ -309,6 +309,6 @@
     <axis
       xyz="0 0 -1" />
-    <dynamics damping="50.0" friction="5.3"/>
-    <limit effort="53.0" velocity="0.2"/>
+    <dynamics damping="50.0" friction="2.7"/>
+    <limit effort="73.0" velocity="0.2"/>
   </joint>
   <transmission name="prox_pitch_transmission">
@@ -385,6 +385,6 @@
     <axis
       xyz="0 0 1" />
-    <dynamics damping="50.0" friction="0.6"/>
-    <limit effort="5.7" velocity="0.2" />
+    <dynamics damping="50.0" friction="0.3"/>
+    <limit effort="25.7" velocity="0.2" />
   </joint>
   <transmission name="dist_pitch_transmission">
@@ -470,6 +470,6 @@
     <axis
       xyz="0 0 -1" />
-    <dynamics damping="50.0" friction="0.6"/>
-    <limit effort="5.7" velocity="0.2" />
+    <dynamics damping="50.0" friction="0.3"/>
+    <limit effort="25.7" velocity="0.2" />
   </joint>
   <transmission name="hand_yaw_transmission">
@@ -574,6 +574,6 @@
     <axis
       xyz="0 0 -1" />
-    <dynamics damping="50.0" friction="1.0"/>
-    <limit effort="10.0" velocity="0.2" />
+    <dynamics damping="50.0" friction="0.5"/>
+    <limit effort="20.0" velocity="0.2" />
   </joint>
   <transmission name="scoop_yaw_transmission">

Commit message: Changed joints damping value for stability at 160Hz

File: ow_lander/urdf/lander.xacro (robot description, xacro)
@@ -157,5 +157,5 @@
     <axis
       xyz="0 0 -1" />
-    <dynamics damping="50.0" friction="2.6"/>
+    <dynamics damping="9.0" friction="2.6"/>
     <limit effort="70.9" velocity="0.15" lower="-1.8" upper="1.8"/>
   </joint>
@@ -233,5 +233,5 @@
     <axis
       xyz="0 0 -1" />
-    <dynamics damping="50.0" friction="4.6"/>
+    <dynamics damping="9.0" friction="4.6"/>
     <limit effort="101.0" velocity="0.2" lower="0.05" upper="2.2"/>
   </joint>
@@ -309,5 +309,5 @@
     <axis
       xyz="0 0 -1" />
-    <dynamics damping="50.0" friction="2.7"/>
+    <dynamics damping="9.0" friction="2.7"/>
     <limit effort="73.0" velocity="0.2"/>
   </joint>
@@ -385,5 +385,5 @@
     <axis
       xyz="0 0 1" />
-    <dynamics damping="50.0" friction="0.3"/>
+    <dynamics damping="9.0" friction="0.3"/>
     <limit effort="25.7" velocity="0.2" />
   </joint>
@@ -470,5 +470,5 @@
     <axis
       xyz="0 0 -1" />
-    <dynamics damping="50.0" friction="0.3"/>
+    <dynamics damping="9.0" friction="0.3"/>
     <limit effort="25.7" velocity="0.2" />
   </joint>
@@ -574,5 +574,5 @@
     <axis
       xyz="0 0 -1" />
-    <dynamics damping="50.0" friction="0.5"/>
+    <dynamics damping="9.0" friction="0.5"/>
     <limit effort="20.0" velocity="0.2" />
   </joint>

Commit message: Reverted changes introduced in the last commit for merging this branch

File: ow_lander/urdf/lander.xacro (robot description, xacro)
@@ -157,5 +157,5 @@
     <axis
       xyz="0 0 -1" />
-    <dynamics damping="9.0" friction="2.6"/>
+    <dynamics damping="50.0" friction="2.6"/>
     <limit effort="70.9" velocity="0.15" lower="-1.8" upper="1.8"/>
   </joint>
@@ -233,5 +233,5 @@
     <axis
       xyz="0 0 -1" />
-    <dynamics damping="9.0" friction="4.6"/>
+    <dynamics damping="50.0" friction="4.6"/>
     <limit effort="101.0" velocity="0.2" lower="0.05" upper="2.2"/>
   </joint>
@@ -309,5 +309,5 @@
     <axis
       xyz="0 0 -1" />
-    <dynamics damping="9.0" friction="2.7"/>
+    <dynamics damping="50.0" friction="2.7"/>
     <limit effort="73.0" velocity="0.2"/>
   </joint>
@@ -385,5 +385,5 @@
     <axis
       xyz="0 0 1" />
-    <dynamics damping="9.0" friction="0.3"/>
+    <dynamics damping="50.0" friction="0.3"/>
     <limit effort="25.7" velocity="0.2" />
   </joint>
@@ -470,5 +470,5 @@
     <axis
       xyz="0 0 -1" />
-    <dynamics damping="9.0" friction="0.3"/>
+    <dynamics damping="50.0" friction="0.3"/>
     <limit effort="25.7" velocity="0.2" />
   </joint>
@@ -574,5 +574,5 @@
     <axis
       xyz="0 0 -1" />
-    <dynamics damping="9.0" friction="0.5"/>
+    <dynamics damping="50.0" friction="0.5"/>
     <limit effort="20.0" velocity="0.2" />
   </joint>

Commit message: Antenna: added realistic maximum effort and velocity, damping values. Tuned PID.

File: ow_lander/urdf/lander.xacro (robot description, xacro)
@@ -728,6 +728,6 @@
     <axis
       xyz="0 0 -1" />
-    <dynamics damping="50" />
-    <limit effort="1000.0" velocity="0.4" />
+    <dynamics damping="10.0" />
+    <limit effort="80.0" velocity="0.2" />
   </joint>
   <transmission name="ant_pan_transmission">
@@ -804,6 +804,6 @@
     <axis
       xyz="0 0 -1" />
-    <dynamics damping="50" />
-    <limit effort="1000.0" velocity="0.4" />
+    <dynamics damping="10.0" />
+    <limit effort="100.0" velocity="0.2" />
   </joint>
   <transmission name="ant_tilt_transmission">

Commit message: Changed grinder collision model to combination of co-axial cylinders

File: ow_lander/urdf/lander.xacro (robot description, xacro)
@@ -610,16 +610,47 @@
       </geometry>
       <material
-        name="">
-        <color
-          rgba="0.6 0.6 0.6 1" />
-      </material>
-    </visual>
-    <collision>
-      <origin
-        xyz="0 0 0"
-        rpy="0 0 0" />
-      <geometry>
-        <mesh
-          filename="package://ow_lander/meshes/l_grinder.STL" />
+       name="">
+       <color
+         rgba="0.6 0.6 0.6 1" />
+     </material>
+    </visual>
+    <collision>
+      <origin
+        xyz="0.08 0 0"
+        rpy="1.57 1.57 1.57" />
+      <geometry>
+        <cylinder radius="0.04" length="0.16"/>
+      </geometry>
+    </collision>
+    <collision>
+      <origin
+        xyz="0.06 0 0"
+        rpy="1.57 1.57 1.57" />
+      <geometry>
+        <cylinder radius="0.05" length="0.12"/>
+      </geometry>
+    </collision>
+    <collision>
+      <origin
+        xyz="0.04 0 0"
+        rpy="1.57 1.57 1.57" />
+      <geometry>
+        <cylinder radius="0.06" length="0.08"/>
+      </geometry>
+    </collision>
+    <collision>
+      <origin
+        xyz="0.02 0 0"
+        rpy="1.57 1.57 1.57" />
+      <geometry>
+        <cylinder radius="0.07" length="0.04"/>
+      </geometry>
+    </collision>
+    <collision>
+      <origin
+        xyz="0.005 0 0"
+        rpy="1.57 1.57 1.57" />
+      <geometry>
+        <cylinder radius="0.075" length="0.01"/>
       </geometry>
     </collision>

Commit message: Reduced joints damping. For scoop collision: removed kp, reduced kd, reduced max_contact_points

File: ow_lander/urdf/lander.xacro (robot description, xacro)
@@ -157,5 +157,5 @@
     <axis
       xyz="0 0 -1" />
-    <dynamics damping="50.0" friction="2.6"/>
+    <dynamics damping="10.0" friction="2.6"/>
     <limit effort="70.9" velocity="0.15" lower="-1.8" upper="1.8"/>
   </joint>
@@ -233,5 +233,5 @@
     <axis
       xyz="0 0 -1" />
-    <dynamics damping="50.0" friction="4.6"/>
+    <dynamics damping="10.0" friction="4.6"/>
     <limit effort="101.0" velocity="0.2" lower="0.05" upper="2.2"/>
   </joint>
@@ -309,5 +309,5 @@
     <axis
       xyz="0 0 -1" />
-    <dynamics damping="50.0" friction="2.7"/>
+    <dynamics damping="10.0" friction="2.7"/>
     <limit effort="73.0" velocity="0.2"/>
   </joint>
@@ -385,5 +385,5 @@
     <axis
       xyz="0 0 1" />
-    <dynamics damping="50.0" friction="0.3"/>
+    <dynamics damping="10.0" friction="0.3"/>
     <limit effort="25.7" velocity="0.2" />
   </joint>
@@ -470,5 +470,5 @@
     <axis
       xyz="0 0 -1" />
-    <dynamics damping="50.0" friction="0.3"/>
+    <dynamics damping="10.0" friction="0.3"/>
     <limit effort="25.7" velocity="0.2" />
   </joint>
@@ -534,10 +534,10 @@
     <selfCollide>1</selfCollide>
     <collision>
+      <max_contacts>1</max_contacts>
       <surface>
         <contact>
           <collide_bitmask>0x0001</collide_bitmask> <!-- Enable collision with the terrain by matching the bitmask -->
           <ode>
-            <kp>1e+15</kp>
-            <kd>1e+13</kd>
+            <kd>5e11</kd>
           </ode>
         </contact>
@@ -574,5 +574,5 @@
     <axis
       xyz="0 0 -1" />
-    <dynamics damping="50.0" friction="0.5"/>
+    <dynamics damping="10.0" friction="0.5"/>
     <limit effort="20.0" velocity="0.2" />
   </joint>

Commit message: Lnader Xacro File Tuning

File: ow_lander/urdf/lander.xacro (robot description, xacro)
@@ -157,5 +157,5 @@
     <axis
       xyz="0 0 -1" />
-    <dynamics damping="50.0" friction="2.6"/>
+    <dynamics damping="10.0" friction="2.6"/>
     <limit effort="70.9" velocity="0.15" lower="-1.8" upper="1.8"/>
   </joint>
@@ -233,5 +233,5 @@
     <axis
       xyz="0 0 -1" />
-    <dynamics damping="50.0" friction="4.6"/>
+    <dynamics damping="10.0" friction="4.6"/>
     <limit effort="101.0" velocity="0.2" lower="0.05" upper="2.2"/>
   </joint>
@@ -309,5 +309,5 @@
     <axis
       xyz="0 0 -1" />
-    <dynamics damping="50.0" friction="2.7"/>
+    <dynamics damping="10.0" friction="2.7"/>
     <limit effort="73.0" velocity="0.2"/>
   </joint>
@@ -385,5 +385,5 @@
     <axis
       xyz="0 0 1" />
-    <dynamics damping="50.0" friction="0.3"/>
+    <dynamics damping="10.0" friction="0.3"/>
     <limit effort="25.7" velocity="0.2" />
   </joint>
@@ -470,5 +470,5 @@
     <axis
       xyz="0 0 -1" />
-    <dynamics damping="50.0" friction="0.3"/>
+    <dynamics damping="10.0" friction="0.3"/>
     <limit effort="25.7" velocity="0.2" />
   </joint>
@@ -538,6 +538,5 @@
           <collide_bitmask>0x0001</collide_bitmask> <!-- Enable collision with the terrain by matching the bitmask -->
           <ode>
-            <kp>1e+15</kp>
-            <kd>1e+13</kd>
+            <kd>1e12</kd>
           </ode>
         </contact>
@@ -574,5 +573,5 @@
     <axis
       xyz="0 0 -1" />
-    <dynamics damping="50.0" friction="0.5"/>
+    <dynamics damping="10.0" friction="0.5"/>
     <limit effort="20.0" velocity="0.2" />
   </joint>
@@ -610,16 +609,47 @@
       </geometry>
       <material
-        name="">
-        <color
-          rgba="0.6 0.6 0.6 1" />
-      </material>
-    </visual>
-    <collision>
-      <origin
-        xyz="0 0 0"
-        rpy="0 0 0" />
-      <geometry>
-        <mesh
-          filename="package://ow_lander/meshes/l_grinder.STL" />
+       name="">
+       <color
+         rgba="0.6 0.6 0.6 1" />
+     </material>
+    </visual>
+    <collision>
+      <origin
+        xyz="0.08 0 0"
+        rpy="1.57 1.57 1.57" />
+      <geometry>
+        <cylinder radius="0.04" length="0.16"/>
+      </geometry>
+    </collision>
+    <collision>
+      <origin
+        xyz="0.06 0 0"
+        rpy="1.57 1.57 1.57" />
+      <geometry>
+        <cylinder radius="0.05" length="0.12"/>
+      </geometry>
+    </collision>
+    <collision>
+      <origin
+        xyz="0.04 0 0"
+        rpy="1.57 1.57 1.57" />
+      <geometry>
+        <cylinder radius="0.06" length="0.08"/>
+      </geometry>
+    </collision>
+    <collision>
+      <origin
+        xyz="0.02 0 0"
+        rpy="1.57 1.57 1.57" />
+      <geometry>
+        <cylinder radius="0.07" length="0.04"/>
+      </geometry>
+    </collision>
+    <collision>
+      <origin
+        xyz="0.005 0 0"
+        rpy="1.57 1.57 1.57" />
+      <geometry>
+        <cylinder radius="0.075" length="0.01"/>
       </geometry>
     </collision>
@@ -641,4 +671,8 @@
         <contact>
           <collide_bitmask>0x0001</collide_bitmask> <!-- Enable collision with the terrain by matching the bitmask -->
+          <ode>
+            <kp>1e+10</kp>
+            <kd>1e+10</kd>
+          </ode>
         </contact>
       </surface>
@@ -728,6 +762,6 @@
     <axis
       xyz="0 0 -1" />
-    <dynamics damping="50" />
-    <limit effort="1000.0" velocity="0.4" />
+    <dynamics damping="10.0" />
+    <limit effort="80.0" velocity="0.2" />
   </joint>
   <transmission name="ant_pan_transmission">
@@ -804,6 +838,6 @@
     <axis
       xyz="0 0 -1" />
-    <dynamics damping="50" />
-    <limit effort="1000.0" velocity="0.4" />
+    <dynamics damping="10.0" />
+    <limit effort="100.0" velocity="0.2" />
   </joint>
   <transmission name="ant_tilt_transmission">

Commit message: Revise joint damping values to 50

File: ow_lander/urdf/lander.xacro (robot description, xacro)
@@ -157,5 +157,5 @@
     <axis
       xyz="0 0 -1" />
-    <dynamics damping="10.0" friction="2.6"/>
+    <dynamics damping="50.0" friction="2.6"/>
     <limit effort="70.9" velocity="0.15" lower="-1.8" upper="1.8"/>
   </joint>
@@ -233,5 +233,5 @@
     <axis
       xyz="0 0 -1" />
-    <dynamics damping="10.0" friction="4.6"/>
+    <dynamics damping="50.0" friction="4.6"/>
     <limit effort="101.0" velocity="0.2" lower="0.05" upper="2.2"/>
   </joint>
@@ -309,5 +309,5 @@
     <axis
       xyz="0 0 -1" />
-    <dynamics damping="10.0" friction="2.7"/>
+    <dynamics damping="50.0" friction="2.7"/>
     <limit effort="73.0" velocity="0.2"/>
   </joint>
@@ -385,5 +385,5 @@
     <axis
       xyz="0 0 1" />
-    <dynamics damping="10.0" friction="0.3"/>
+    <dynamics damping="50.0" friction="0.3"/>
     <limit effort="25.7" velocity="0.2" />
   </joint>
@@ -470,5 +470,5 @@
     <axis
       xyz="0 0 -1" />
-    <dynamics damping="10.0" friction="0.3"/>
+    <dynamics damping="50.0" friction="0.3"/>
     <limit effort="25.7" velocity="0.2" />
   </joint>
@@ -573,5 +573,5 @@
     <axis
       xyz="0 0 -1" />
-    <dynamics damping="10.0" friction="0.5"/>
+    <dynamics damping="50.0" friction="0.5"/>
     <limit effort="20.0" velocity="0.2" />
   </joint>
@@ -762,5 +762,5 @@
     <axis
       xyz="0 0 -1" />
-    <dynamics damping="10.0" />
+    <dynamics damping="50.0" />
     <limit effort="80.0" velocity="0.2" />
   </joint>
@@ -838,5 +838,5 @@
     <axis
       xyz="0 0 -1" />
-    <dynamics damping="10.0" />
+    <dynamics damping="50.0" />
     <limit effort="100.0" velocity="0.2" />
   </joint>
