Commit message: Sharing my branch with Ussama so he can work on it

File: ow_lander/urdf/lander.xacro (robot description, xacro)
@@ -157,5 +157,5 @@
     <axis
       xyz="0 0 -1" />
-    <dynamics damping="50.0" friction="2.6"/>
+    <dynamics damping="1.0" friction="2.6"/>
     <limit effort="70.9" velocity="0.15" lower="-1.8" upper="1.8"/>
   </joint>
@@ -233,5 +233,5 @@
     <axis
       xyz="0 0 -1" />
-    <dynamics damping="50.0" friction="4.6"/>
+    <dynamics damping="1.0" friction="4.6"/>
     <limit effort="101.0" velocity="0.2" lower="0.05" upper="2.2"/>
   </joint>
@@ -309,5 +309,5 @@
     <axis
       xyz="0 0 -1" />
-    <dynamics damping="50.0" friction="2.7"/>
+    <dynamics damping="1.0" friction="2.7"/>
     <limit effort="73.0" velocity="0.2"/>
   </joint>
@@ -385,5 +385,5 @@
     <axis
       xyz="0 0 1" />
-    <dynamics damping="50.0" friction="0.3"/>
+    <dynamics damping="1.0" friction="0.3"/>
     <limit effort="25.7" velocity="0.2" />
   </joint>
@@ -470,5 +470,5 @@
     <axis
       xyz="0 0 -1" />
-    <dynamics damping="50.0" friction="0.3"/>
+    <dynamics damping="1.0" friction="0.3"/>
     <limit effort="25.7" velocity="0.2" />
   </joint>
@@ -573,5 +573,5 @@
     <axis
       xyz="0 0 -1" />
-    <dynamics damping="50.0" friction="0.5"/>
+    <dynamics damping="1.0" friction="0.5"/>
     <limit effort="20.0" velocity="0.2" />
   </joint>
@@ -686,6 +686,6 @@
     <child link="l_grinder" />
     <axis xyz="-1 0 0" />
-    <dynamics damping="1" />
-    <limit lower="-3.14" upper="3.14" effort="1.0" velocity="0.1" />
+    <dynamics damping="0.01" />
+    <limit lower="-3.14" upper="3.14" effort="20.0" velocity="0.3" />
   </joint>
   <transmission name="grinder_yaw_transmission">

Commit message: Rebuilt the scoop's collider with cubes that approximate its shape.

File: ow_lander/urdf/lander.xacro (robot description, xacro)
@@ -523,11 +523,47 @@
       </material>
     </visual>
-    <collision>
-      <origin
-        xyz="0 0 0"
-        rpy="0 0 0" />
-      <geometry>
-        <mesh
-          filename="package://ow_lander/meshes/l_scoop.STL" />
+    <!-- scoop bottom -->
+    <collision>
+      <origin
+        xyz="0.030115 0 0.076505"
+        rpy="0 -0.0349040838 0" />
+      <geometry>
+          <box size="0.1273 0.0818 0.002"/>
+      </geometry>
+    </collision>
+    <!-- scoop backing (flat) -->
+    <collision>
+      <origin
+        xyz="-0.032195 0 0.036854"
+        rpy="0 -1.60570041059 0" />
+      <geometry>
+          <box size="0.0749 0.0818 0.002"/>
+      </geometry>
+    </collision>
+    <!-- scoop left sidewall -->
+    <collision>
+      <origin
+        xyz="0.025676 -0.0409 0.038875"
+        rpy="1.5708 -0.0349040838 0" />
+      <geometry>
+          <box size="0.1158 0.0749 0.002"/>
+      </geometry>
+    </collision>
+    <!-- scoop right sidewall -->
+    <collision>
+      <origin
+        xyz="0.025676 0.0409 0.038875"
+        rpy="1.5708 -0.0349040838 0" />
+      <geometry>
+          <box size="0.1158 0.0749 0.002"/>
+      </geometry>
+    </collision>
+    <!-- scoop top -->
+    <collision>
+      <origin
+        xyz="0.000264 0 0.000512"
+        rpy="0 -0.0349040838 0" />
+      <geometry>
+          <box size="0.06234 0.0818 0.002"/>
       </geometry>
     </collision>

Commit message: Added colliders for the tip of the scoop

File: ow_lander/urdf/lander.xacro (robot description, xacro)
@@ -566,4 +566,22 @@
       <geometry>
           <box size="0.06234 0.0818 0.002"/>
+      </geometry>
+    </collision>
+    <!-- scoop wide tip -->
+    <collision>
+      <origin
+        xyz="0.090908 0 0.079513"
+        rpy="0 -0.254542712 0" />
+      <geometry>
+          <box size="0.008122 0.0818 0.002"/>
+      </geometry>
+    </collision>
+    <!-- scoop wide tip -->
+    <collision>
+      <origin
+        xyz="0.092572 0 0.079946"
+        rpy="0 -0.254542712 0" />
+      <geometry>
+          <box size="0.01156 0.04346 0.001"/>
       </geometry>
     </collision>

Commit message: disabled collions for debugging

File: ow_lander/urdf/lander.xacro (robot description, xacro)
@@ -523,5 +523,5 @@
       </material>
     </visual>
-    <collision>
+    <!--collision>
       <origin
         xyz="0 0 0"
@@ -531,5 +531,5 @@
           filename="package://ow_lander/meshes/l_scoop.STL" />
       </geometry>
-    </collision>
+    </collision-->
   </link>
   <gazebo reference="l_scoop">
@@ -626,5 +626,5 @@
      </material>
     </visual>
-    <collision>
+    <!--collision>
       <origin
         xyz="0.08 0 0"
@@ -665,5 +665,5 @@
         <cylinder radius="0.075" length="0.01"/>
       </geometry>
-    </collision>
+    </collision-->
   </link>
   <gazebo reference="l_grinder">
@@ -679,8 +679,8 @@
     </visual>
     <selfCollide>1</selfCollide>
-    <collision>
+    <!--collision>
       <surface>
         <contact>
-          <collide_bitmask>0x0001</collide_bitmask> <!-- Enable collision with the terrain by matching the bitmask -->
+          <collide_bitmask>0x0001</collide_bitmask> <Enable collision with the terrain by matching the bitmask>
           <ode>
             <kp>1e+10</kp>
@@ -689,5 +689,5 @@
         </contact>
       </surface>
-    </collision>
+    </collision-->
   </gazebo>
   <joint

Commit message: working copy of with native linux 1804

File: ow_lander/urdf/lander.xacro (robot description, xacro)
@@ -158,5 +158,5 @@
       xyz="0 0 -1" />
     <dynamics damping="50.0" friction="2.6"/>
-    <limit effort="70.9" velocity="0.15" lower="-1.8" upper="1.8"/>
+    <limit effort="70.9" velocity="1.0" lower="-1.8" upper="1.8"/>
   </joint>
   <transmission name="shou_yaw_transmission">
@@ -234,5 +234,5 @@
       xyz="0 0 -1" />
     <dynamics damping="50.0" friction="4.6"/>
-    <limit effort="101.0" velocity="0.2" lower="0.05" upper="2.2"/>
+    <limit effort="101.0" velocity="1.0" lower="0.05" upper="2.2"/>
   </joint>
   <transmission name="shou_pitch_transmission">
@@ -310,5 +310,5 @@
       xyz="0 0 -1" />
     <dynamics damping="50.0" friction="2.7"/>
-    <limit effort="73.0" velocity="0.2"/>
+    <limit effort="73.0" velocity="1.0"/>
   </joint>
   <transmission name="prox_pitch_transmission">
@@ -386,5 +386,5 @@
       xyz="0 0 1" />
     <dynamics damping="50.0" friction="0.3"/>
-    <limit effort="25.7" velocity="0.2" />
+    <limit effort="25.7" velocity="1.0" />
   </joint>
   <transmission name="dist_pitch_transmission">
@@ -483,5 +483,5 @@
       xyz="0 0 -1" />
     <dynamics damping="50.0" friction="0.3"/>
-    <limit effort="25.7" velocity="0.2" />
+    <limit effort="25.7" velocity="1.0" />
   </joint>
   <transmission name="hand_yaw_transmission">
@@ -586,5 +586,5 @@
       xyz="0 0 -1" />
     <dynamics damping="50.0" friction="0.5"/>
-    <limit effort="20.0" velocity="0.2" />
+    <limit effort="20.0" velocity="1.0" />
   </joint>
   <transmission name="scoop_yaw_transmission">
@@ -699,5 +699,5 @@
     <axis xyz="-1 0 0" />
     <dynamics damping="1" />
-    <limit lower="-3.14" upper="3.14" effort="1.0" velocity="0.1" />
+    <limit lower="-3.14" upper="3.14" effort="1.0" velocity="1.0" />
   </joint>
   <transmission name="grinder_yaw_transmission">
@@ -775,6 +775,6 @@
       xyz="0 0 -1" />
     <dynamics damping="50.0" />
-    <limit effort="80.0" velocity="0.2" />
-  </joint>
+    <limit effort="80.0" velocity="1.0" />
+  </joint>                         0
   <transmission name="ant_pan_transmission">
     <type>transmission_interface/SimpleTransmission</type>
@@ -851,5 +851,5 @@
       xyz="0 0 -1" />
     <dynamics damping="50.0" />
-    <limit effort="100.0" velocity="0.2" />
+    <limit effort="100.0" velocity="1.0" />
   </joint>
   <transmission name="ant_tilt_transmission">

Commit message: fixing velocity limits in both joint_limit.yamls and lander.xarco file

File: ow_lander/urdf/lander.xacro (robot description, xacro)
@@ -158,5 +158,5 @@
       xyz="0 0 -1" />
     <dynamics damping="50.0" friction="2.6"/>
-    <limit effort="70.9" velocity="0.15" lower="-1.8" upper="1.8"/>
+    <limit effort="70.9" velocity="1.0" lower="-1.8" upper="1.8"/>
   </joint>
   <transmission name="shou_yaw_transmission">
@@ -234,5 +234,5 @@
       xyz="0 0 -1" />
     <dynamics damping="50.0" friction="4.6"/>
-    <limit effort="101.0" velocity="0.2" lower="0.05" upper="2.2"/>
+    <limit effort="101.0" velocity="1.0" lower="0.05" upper="2.2"/>
   </joint>
   <transmission name="shou_pitch_transmission">
@@ -310,5 +310,5 @@
       xyz="0 0 -1" />
     <dynamics damping="50.0" friction="2.7"/>
-    <limit effort="73.0" velocity="0.2"/>
+    <limit effort="73.0" velocity="1.0"/>
   </joint>
   <transmission name="prox_pitch_transmission">
@@ -386,5 +386,5 @@
       xyz="0 0 1" />
     <dynamics damping="50.0" friction="0.3"/>
-    <limit effort="25.7" velocity="0.2" />
+    <limit effort="25.7" velocity="1.0" />
   </joint>
   <transmission name="dist_pitch_transmission">
@@ -483,5 +483,5 @@
       xyz="0 0 -1" />
     <dynamics damping="50.0" friction="0.3"/>
-    <limit effort="25.7" velocity="0.2" />
+    <limit effort="25.7" velocity="1.0" />
   </joint>
   <transmission name="hand_yaw_transmission">
@@ -586,5 +586,5 @@
       xyz="0 0 -1" />
     <dynamics damping="50.0" friction="0.5"/>
-    <limit effort="20.0" velocity="0.2" />
+    <limit effort="20.0" velocity="1.0" />
   </joint>
   <transmission name="scoop_yaw_transmission">
@@ -699,5 +699,5 @@
     <axis xyz="-1 0 0" />
     <dynamics damping="1" />
-    <limit lower="-3.14" upper="3.14" effort="1.0" velocity="0.1" />
+    <limit lower="-3.14" upper="3.14" effort="1.0" velocity="1.0" />
   </joint>
   <transmission name="grinder_yaw_transmission">
@@ -775,5 +775,5 @@
       xyz="0 0 -1" />
     <dynamics damping="50.0" />
-    <limit effort="80.0" velocity="0.2" />
+    <limit effort="80.0" velocity="1.0" />
   </joint>
   <transmission name="ant_pan_transmission">
@@ -851,5 +851,5 @@
       xyz="0 0 -1" />
     <dynamics damping="50.0" />
-    <limit effort="100.0" velocity="0.2" />
+    <limit effort="100.0" velocity="1.0" />
   </joint>
   <transmission name="ant_tilt_transmission">

Commit message: Quick prototype of Joints Locking feature

File: ow_lander/urdf/lander.xacro (robot description, xacro)
@@ -818,5 +818,5 @@
   <joint
     name="j_ant_pan"
-    type="continuous">
+    type="revolute">
     <origin
       xyz="0 0.58 0.675"
@@ -829,5 +829,5 @@
       xyz="0 0 -1" />
     <dynamics damping="50.0" />
-    <limit effort="80.0" velocity="0.2" />
+    <limit effort="80.0" velocity="0.2" lower="-3.14" upper="3.14" />
   </joint>
   <transmission name="ant_pan_transmission">
@@ -894,5 +894,5 @@
   <joint
     name="j_ant_tilt"
-    type="continuous">
+    type="revolute">
     <origin
       xyz="0 0 -0.24805"
@@ -905,5 +905,5 @@
       xyz="0 0 -1" />
     <dynamics damping="50.0" />
-    <limit effort="100.0" velocity="0.2" />
+    <limit effort="100.0" velocity="0.2" lower="-1.5" upper="1.5" />
   </joint>
   <transmission name="ant_tilt_transmission">
@@ -920,4 +920,7 @@
       <robotNamespace>/</robotNamespace>
     </plugin>
+    <plugin name="ow_faults_joints" filename="libow_faults_joints.so">
+      <robotNamespace>/</robotNamespace>
+    </plugin>
     <!-- Publish joint states so rviz can visualize them. -->
     <!--plugin name="joint_state_publisher" filename="libgazebo_ros_joint_state_publisher.so">

Commit message: remove commented code + increase pan joint limits  + address  other PR comments

File: ow_lander/urdf/lander.xacro (robot description, xacro)
@@ -829,5 +829,5 @@
       xyz="0 0 -1" />
     <dynamics damping="50.0" />
-    <limit effort="80.0" velocity="0.2" lower="-3.14" upper="3.14" />
+    <limit effort="80.0" velocity="0.2" lower="-3.50" upper="3.50" />
   </joint>
   <transmission name="ant_pan_transmission">

Commit message: convert all continuous joints to revolute with large up/down limits

File: ow_lander/urdf/lander.xacro (robot description, xacro)
@@ -299,5 +299,5 @@
   <joint
     name="j_prox_pitch"
-    type="continuous">
+    type="revolute">
     <origin
       xyz="0.53 0 0"
@@ -310,5 +310,5 @@
       xyz="0 0 -1" />
     <dynamics damping="50.0" friction="2.7"/>
-    <limit effort="73.0" velocity="0.2"/>
+    <limit effort="73.0" velocity="0.2" lower="1000000" upper="1000000"/>
   </joint>
   <transmission name="prox_pitch_transmission">
@@ -375,5 +375,5 @@
   <joint
     name="j_dist_pitch"
-    type="continuous">
+    type="revolute">
     <origin
       xyz="0.586 0 -0.15"
@@ -386,5 +386,5 @@
       xyz="0 0 1" />
     <dynamics damping="50.0" friction="0.3"/>
-    <limit effort="25.7" velocity="0.2" />
+    <limit effort="25.7" velocity="0.2" lower="1000000" upper="1000000"/>
   </joint>
   <transmission name="dist_pitch_transmission">
@@ -472,5 +472,5 @@
   <joint
     name="j_hand_yaw"
-    type="continuous">
+    type="revolute">
     <origin
       xyz="0.163 0.2 0"
@@ -483,5 +483,5 @@
       xyz="0 0 -1" />
     <dynamics damping="50.0" friction="0.3"/>
-    <limit effort="25.7" velocity="0.2" />
+    <limit effort="25.7" velocity="0.2" lower="1000000" upper="1000000"/>
   </joint>
   <transmission name="hand_yaw_transmission">
@@ -629,5 +629,5 @@
   <joint
     name="j_scoop_yaw"
-    type="continuous">
+    type="revolute">
     <origin
       xyz="0.15 0 0"
@@ -640,5 +640,5 @@
       xyz="0 0 -1" />
     <dynamics damping="50.0" friction="0.5"/>
-    <limit effort="20.0" velocity="0.2" />
+    <limit effort="20.0" velocity="0.2" lower="1000000" upper="1000000"/>
   </joint>
   <transmission name="scoop_yaw_transmission">
@@ -753,5 +753,5 @@
     <axis xyz="-1 0 0" />
     <dynamics damping="1" />
-    <limit lower="-3.14" upper="3.14" effort="1.0" velocity="0.1" />
+    <limit effort="1.0" velocity="0.1" lower="-3.14" upper="3.14"/>
   </joint>
   <transmission name="grinder_yaw_transmission">

Commit message: correct the signs

File: ow_lander/urdf/lander.xacro (robot description, xacro)
@@ -310,5 +310,5 @@
       xyz="0 0 -1" />
     <dynamics damping="50.0" friction="2.7"/>
-    <limit effort="73.0" velocity="0.2" lower="1000000" upper="1000000"/>
+    <limit effort="73.0" velocity="0.2" lower="-1000000" upper="1000000"/>
   </joint>
   <transmission name="prox_pitch_transmission">
@@ -386,5 +386,5 @@
       xyz="0 0 1" />
     <dynamics damping="50.0" friction="0.3"/>
-    <limit effort="25.7" velocity="0.2" lower="1000000" upper="1000000"/>
+    <limit effort="25.7" velocity="0.2" lower="-1000000" upper="1000000"/>
   </joint>
   <transmission name="dist_pitch_transmission">
@@ -483,5 +483,5 @@
       xyz="0 0 -1" />
     <dynamics damping="50.0" friction="0.3"/>
-    <limit effort="25.7" velocity="0.2" lower="1000000" upper="1000000"/>
+    <limit effort="25.7" velocity="0.2" lower="-1000000" upper="1000000"/>
   </joint>
   <transmission name="hand_yaw_transmission">
@@ -640,5 +640,5 @@
       xyz="0 0 -1" />
     <dynamics damping="50.0" friction="0.5"/>
-    <limit effort="20.0" velocity="0.2" lower="1000000" upper="1000000"/>
+    <limit effort="20.0" velocity="0.2" lower="-1000000" upper="1000000"/>
   </joint>
   <transmission name="scoop_yaw_transmission">

Commit message: Reset joint types and switch to using joint friction instead of joints upper/lower limits

File: ow_lander/urdf/lander.xacro (robot description, xacro)
@@ -299,5 +299,5 @@
   <joint
     name="j_prox_pitch"
-    type="revolute">
+    type="continuous">
     <origin
       xyz="0.53 0 0"
@@ -310,5 +310,5 @@
       xyz="0 0 -1" />
     <dynamics damping="50.0" friction="2.7"/>
-    <limit effort="73.0" velocity="0.2" lower="-1000000" upper="1000000"/>
+    <limit effort="73.0" velocity="0.2"/>
   </joint>
   <transmission name="prox_pitch_transmission">
@@ -375,5 +375,5 @@
   <joint
     name="j_dist_pitch"
-    type="revolute">
+    type="continuous">
     <origin
       xyz="0.586 0 -0.15"
@@ -386,5 +386,5 @@
       xyz="0 0 1" />
     <dynamics damping="50.0" friction="0.3"/>
-    <limit effort="25.7" velocity="0.2" lower="-1000000" upper="1000000"/>
+    <limit effort="25.7" velocity="0.2" />
   </joint>
   <transmission name="dist_pitch_transmission">
@@ -472,5 +472,5 @@
   <joint
     name="j_hand_yaw"
-    type="revolute">
+    type="continuous">
     <origin
       xyz="0.163 0.2 0"
@@ -483,5 +483,5 @@
       xyz="0 0 -1" />
     <dynamics damping="50.0" friction="0.3"/>
-    <limit effort="25.7" velocity="0.2" lower="-1000000" upper="1000000"/>
+    <limit effort="25.7" velocity="0.2" />
   </joint>
   <transmission name="hand_yaw_transmission">
@@ -629,5 +629,5 @@
   <joint
     name="j_scoop_yaw"
-    type="revolute">
+    type="continuous">
     <origin
       xyz="0.15 0 0"
@@ -640,5 +640,5 @@
       xyz="0 0 -1" />
     <dynamics damping="50.0" friction="0.5"/>
-    <limit effort="20.0" velocity="0.2" lower="-1000000" upper="1000000"/>
+    <limit effort="20.0" velocity="0.2" />
   </joint>
   <transmission name="scoop_yaw_transmission">

Commit message: revert antenna joints types to continuous

File: ow_lander/urdf/lander.xacro (robot description, xacro)
@@ -818,5 +818,5 @@
   <joint
     name="j_ant_pan"
-    type="revolute">
+    type="continuous">
     <origin
       xyz="0 0.58 0.675"
@@ -829,5 +829,5 @@
       xyz="0 0 -1" />
     <dynamics damping="50.0" />
-    <limit effort="80.0" velocity="0.2" lower="-3.50" upper="3.50" />
+    <limit effort="80.0" velocity="0.2" />
   </joint>
   <transmission name="ant_pan_transmission">
@@ -894,5 +894,5 @@
   <joint
     name="j_ant_tilt"
-    type="revolute">
+    type="continuous">
     <origin
       xyz="0 0 -0.24805"
@@ -905,5 +905,5 @@
       xyz="0 0 -1" />
     <dynamics damping="50.0" />
-    <limit effort="100.0" velocity="0.2" lower="-1.5" upper="1.5" />
+    <limit effort="100.0" velocity="0.2" />
   </joint>
   <transmission name="ant_tilt_transmission">

Commit message: simple ingest sample action implemented

File: ow_lander/urdf/lander.xacro (robot description, xacro)
@@ -17,5 +17,5 @@
   <xacro:include filename="$(find ow_lander)/urdf/lander_sample_dock.xacro" />
   <xacro:lander_sample_dock lander_sample_dock_parent_link="base_link"
-                     off_x="0.53" off_y="-0.35" off_z="0.32" off_R="-${pi/2.0}" off_P="0.0" off_Y="-${pi/2.0}"
+                     off_x="0.5226" off_y="-0.35" off_z="0.32" off_R="-${pi/2.0}" off_P="0.0" off_Y="-${pi/2.0}"
                      vis_mask="${vis_mask}" />
   <xacro:arg name="freeze_base_link" default="false"/>

File: ow_lander/urdf/lander_sample_dock.xacro (robot description, xacro)
@@ -63,4 +63,17 @@
         </plugin>
       </visual>
+      <sensor name="contact_sensor_sample_dock" type="contact">
+        <parent link="lander_sample_dock${suffix}"/>
+        <contact>
+          <collision>
+            lander_sample_dock_link_fixed_joint_lump__lander_sample_dock${suffix}_collision
+          </collision>
+        </contact>
+        <plugin name="contact_sensor_sample_dock_plugin"
+                filename="libContactSensorPlugin.so">
+          <topic>/ow_regolith/contacts/sample_dock</topic>
+          <report_only>regolith_\d*.*</report_only>
+        </plugin>
+      </sensor>
     </gazebo>
   </xacro:macro>

Commit message: intial commit with safe margins

File: ow_lander/urdf/lander.xacro (robot description, xacro)
@@ -310,5 +310,5 @@
       xyz="0 0 -1" />
     <dynamics damping="50.0" friction="2.7"/>
-    <limit effort="73.0" velocity="0.2"/>
+    <limit effort="73.0" velocity="0.2" lower="-3.14" upper="3.14"/>
   </joint>
   <transmission name="prox_pitch_transmission">
@@ -386,5 +386,5 @@
       xyz="0 0 1" />
     <dynamics damping="50.0" friction="0.3"/>
-    <limit effort="25.7" velocity="0.2" />
+    <limit effort="25.7" velocity="0.2" lower="-3.14" upper="3.14" />
   </joint>
   <transmission name="dist_pitch_transmission">
@@ -483,5 +483,5 @@
       xyz="0 0 -1" />
     <dynamics damping="50.0" friction="0.3"/>
-    <limit effort="25.7" velocity="0.2" />
+    <limit effort="25.7" velocity="0.2" lower="-3.14" upper="3.14"/>
   </joint>
   <transmission name="hand_yaw_transmission">
@@ -640,5 +640,5 @@
       xyz="0 0 -1" />
     <dynamics damping="50.0" friction="0.5"/>
-    <limit effort="20.0" velocity="0.2" />
+    <limit effort="20.0" velocity="0.2" lower="-3.14" upper="3.14"/>
   </joint>
   <transmission name="scoop_yaw_transmission">
@@ -829,5 +829,5 @@
       xyz="0 0 -1" />
     <dynamics damping="50.0" />
-    <limit effort="80.0" velocity="0.2" />
+    <limit effort="80.0" velocity="0.2" lower="-3.14" upper="3.14" />
   </joint>
   <transmission name="ant_pan_transmission">
@@ -905,5 +905,5 @@
       xyz="0 0 -1" />
     <dynamics damping="50.0" />
-    <limit effort="100.0" velocity="0.2" />
+    <limit effort="100.0" velocity="0.2" lower="-3.14" upper="3.14"/>
   </joint>
   <transmission name="ant_tilt_transmission">

Commit message: changing joint limits for shoulder pitch and yaw

File: ow_lander/urdf/lander.xacro (robot description, xacro)
@@ -158,5 +158,5 @@
       xyz="0 0 -1" />
     <dynamics damping="50.0" friction="2.6"/>
-    <limit effort="70.9" velocity="0.15" lower="-1.8" upper="1.8"/>
+    <limit effort="70.9" velocity="0.15" lower="-1.56" upper="1.43"/>
   </joint>
   <transmission name="shou_yaw_transmission">
@@ -234,5 +234,5 @@
       xyz="0 0 -1" />
     <dynamics damping="50.0" friction="4.6"/>
-    <limit effort="101.0" velocity="0.2" lower="0.05" upper="2.2"/>
+    <limit effort="101.0" velocity="0.2" lower="-0.5" upper="2.2"/>
   </joint>
   <transmission name="shou_pitch_transmission">

Commit message: added limits to joints where applicable

File: ow_lander/urdf/lander.xacro (robot description, xacro)
@@ -234,5 +234,5 @@
       xyz="0 0 -1" />
     <dynamics damping="50.0" friction="4.6"/>
-    <limit effort="101.0" velocity="0.2" lower="-0.5" upper="2.2"/>
+    <limit effort="101.0" velocity="0.2" lower="-0.4" upper="2.2"/>
   </joint>
   <transmission name="shou_pitch_transmission">
@@ -386,5 +386,5 @@
       xyz="0 0 1" />
     <dynamics damping="50.0" friction="0.3"/>
-    <limit effort="25.7" velocity="0.2" lower="-3.14" upper="3.14" />
+    <limit effort="25.7" velocity="0.2" lower="-1.9" upper="3.5" />
   </joint>
   <transmission name="dist_pitch_transmission">

Commit message: adding antenna joint limits

File: ow_lander/urdf/lander.xacro (robot description, xacro)
@@ -829,5 +829,5 @@
       xyz="0 0 -1" />
     <dynamics damping="50.0" />
-    <limit effort="80.0" velocity="0.2" lower="-3.14" upper="3.14" />
+    <limit effort="80.0" velocity="0.2" lower="-3.2" upper="3.2" />
   </joint>
   <transmission name="ant_pan_transmission">
@@ -905,5 +905,5 @@
       xyz="0 0 -1" />
     <dynamics damping="50.0" />
-    <limit effort="100.0" velocity="0.2" lower="-3.14" upper="3.14"/>
+    <limit effort="100.0" velocity="0.2" lower="-1.57" upper="1.57"/>
   </joint>
   <transmission name="ant_tilt_transmission">
