Commit message: changing default limits from 3.14 to 3.2

File: ow_lander/urdf/lander.xacro (robot description, xacro)
@@ -310,5 +310,5 @@
       xyz="0 0 -1" />
     <dynamics damping="50.0" friction="2.7"/>
-    <limit effort="73.0" velocity="0.2" lower="-3.14" upper="3.14"/>
+    <limit effort="73.0" velocity="0.2" lower="-3.2" upper="3.2"/>
   </joint>
   <transmission name="prox_pitch_transmission">
@@ -483,5 +483,5 @@
       xyz="0 0 -1" />
     <dynamics damping="50.0" friction="0.3"/>
-    <limit effort="25.7" velocity="0.2" lower="-3.14" upper="3.14"/>
+    <limit effort="25.7" velocity="0.2" lower="-3.2" upper="3.2"/>
   </joint>
   <transmission name="hand_yaw_transmission">
@@ -640,5 +640,5 @@
       xyz="0 0 -1" />
     <dynamics damping="50.0" friction="0.5"/>
-    <limit effort="20.0" velocity="0.2" lower="-3.14" upper="3.14"/>
+    <limit effort="20.0" velocity="0.2" lower="-3.2" upper="3.2"/>
   </joint>
   <transmission name="scoop_yaw_transmission">
@@ -753,5 +753,5 @@
     <axis xyz="-1 0 0" />
     <dynamics damping="1" />
-    <limit effort="1.0" velocity="0.1" lower="-3.14" upper="3.14"/>
+    <limit effort="1.0" velocity="0.1" lower="-3.2" upper="3.2"/>
   </joint>
   <transmission name="grinder_yaw_transmission">

Commit message: chnaging limit of  j_dist_pitch to -2.2 and 3.65.

File: ow_lander/urdf/lander.xacro (robot description, xacro)
@@ -386,5 +386,5 @@
       xyz="0 0 1" />
     <dynamics damping="50.0" friction="0.3"/>
-    <limit effort="25.7" velocity="0.2" lower="-1.9" upper="3.5" />
+    <limit effort="25.7" velocity="0.2" lower="-2.2" upper="3.65" />
   </joint>
   <transmission name="dist_pitch_transmission">

Commit message: Simplified sample dock's definition and placement on lander  - Corrected a weird inertia origin

File: ow_lander/urdf/lander.xacro (robot description, xacro)
@@ -17,5 +17,5 @@
   <xacro:include filename="$(find ow_lander)/urdf/lander_sample_dock.xacro" />
   <xacro:lander_sample_dock lander_sample_dock_parent_link="base_link"
-                     off_x="0.5226" off_y="-0.35" off_z="0.32" off_R="-${pi/2.0}" off_P="0.0" off_Y="-${pi/2.0}"
+                     off_x="0.5476" off_y="-0.35" off_z="0.32" off_R="-${pi/2.0}" off_P="0.0" off_Y="-${pi/2.0}"
                      vis_mask="${vis_mask}" />
   <xacro:arg name="freeze_base_link" default="false"/>

File: ow_lander/urdf/lander_sample_dock.xacro (robot description, xacro)
@@ -24,5 +24,5 @@
     <link name="lander_sample_dock${suffix}">
       <collision>
-        <origin rpy="0 0 0" xyz="0 0 0.025"/>
+        <origin rpy="0 0 0" xyz="0 0 0"/>
         <geometry>
           <mesh filename="package://ow_lander/meshes/sample_dock.stl" />
@@ -30,5 +30,5 @@
       </collision>
       <visual>
-        <origin rpy="0 0 0" xyz="0 0 0.025"/>
+        <origin rpy="0 0 0" xyz="0 0 0.0"/>
         <geometry>
           <mesh filename="package://ow_lander/meshes/sample_dock.stl" />
@@ -39,5 +39,5 @@
       </visual>
       <inertial>
-        <origin rpy="0 0 0" xyz="0 0 0.05"/>
+        <origin rpy="0 0 0" xyz="0 0 0"/>
         <mass value="0.01"/>
         <inertia

Commit message: grinder tip reference link added for precision depth prediction

File: ow_lander/urdf/lander.xacro (robot description, xacro)
@@ -765,4 +765,23 @@
     </actuator>
   </transmission>
+  <!-- link that we can reference in Gazebo to get altitude of tip
+     of grinder above the terrain. Note that without an inertial
+     tag, the link will not show up in the SDF/Gazebo at all -->
+  <link name="l_grinder_tip">
+    <inertial>
+      <mass value="0.0"/>
+      <inertia ixx="0" ixy="0" ixz="0" iyy="0" iyz="0" izz="0"/>
+    </inertial>
+  </link>
+  <joint name="l_grinder_tip_joint" type="fixed">
+    <origin xyz="-0.1550 -0.2684 0.0" rpy="1.5708 1.5708 -0.5236"/>
+    <!-- 1.5708 0 -0.5236 -->
+    <!-- fix to hand so it does not rotate with grinder -->
+    <parent link="l_hand"/>
+    <child link="l_grinder_tip"/>
+  </joint>
+  <gazebo reference="l_grinder_tip_joint">
+    <preserveFixedJoint>true</preserveFixedJoint>
+  </gazebo>
   <link name="l_ant_foot">
     <inertial>

Commit message: TaskGrind redone for more accurate depth

File: ow_lander/urdf/lander.xacro (robot description, xacro)
@@ -775,8 +775,7 @@
   </link>
   <joint name="l_grinder_tip_joint" type="fixed">
-    <origin xyz="-0.1550 -0.2684 0.0" rpy="1.5708 1.5708 -0.5236"/>
-    <!-- 1.5708 0 -0.5236 -->
-    <!-- fix to hand so it does not rotate with grinder -->
-    <parent link="l_hand"/>
+    <origin xyz="0.16 0 0" rpy="0 0 0"/>
+    <parent link="l_grinder"/>
+    <!-- <parent link="l_hand"/> -->
     <child link="l_grinder_tip"/>
   </joint>

Commit message: Fixed tf broadcasting the wrong transform for world -> base_link Arm planning now takes place in the correct frame. Workarounds removed in ow_materials

File: ow_lander/urdf/lander.xacro (robot description, xacro)
@@ -25,4 +25,7 @@
     <link name="world"/>
     <joint name="fixed" type="fixed">
+      <origin
+        xyz="$(arg x) $(arg y) $(arg z)"
+        rpy="$(arg R) $(arg P) $(arg Y)"/>
       <parent link="world"/>
       <child link="base_link"/>
