Commit message: Fix the interpolation between inner-outer radius

File: ow_dynamic_terrain/urdf/simple_camera.urdf (robot description, URDF)
Before this commit: robot pr2, 2 links, 1 joints
Links:
- removed link dummy_link
- added link world
Joints:
- joint dummy_fixed_joint: parent dummy_link -> world
